File: PCB/Barometer.kicad_sch (KiCad schematic)
At the start: 1 part, among them U4 BMP280

Commit message: Updated PCB
Parts:
- added C14, C15: C, symbol PCM_Elektuur:C
Connections:
- net GND: now reaches U4.1 (GND)
- net GND: now also U4.7 (GND), C14.2 (-), C15.2 (-)
- net nCSS_BMP280: now reaches U4.2 (CSB)
- net MISO_BMP280: now reaches U4.3 (SDI)
- net CLK_BMP280: now reaches U4.4 (SCK)
- net MOSI_BMP280: now reaches U4.5 (SDO)
- net +3V3: now reaches U4.6 (VDDIO)
- net +3V3: now also U4.8 (VDD), C14.1 (+), C15.1 (+)
Other:
- moved on the sheet: U4

Commit message: Updated PCB.
Parts:
- renumbered C15 to C1, C14 to C2, U4 to U1
Changed lines of the file:
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@@
 		(dnp no)
 		(fields_autoplaced yes)
-		(property "Reference" "C15"
+		(property "Reference" "C1"
 			(at 127 95.2499 0)
 			(effects
@@
 		(instances
 			(project "IMU_V100"
-				(path "/b6a8d14b-6e32-4628-bf0c-2046877d1cfa/38184d55-d9c0-48fd-bb15-ff1076c43a13"
-					(reference "C15")
+				(path "/b6a8d14b-6e32-4628-bf0c-2046877d1cfa/205555cc-3b86-4915-975e-3a7e3eed6661/33aef508-2230-418a-a3ff-3a2fec798c19"
+					(reference "C1")
 					(unit 1)
 				)
@@
 		(dnp no)
 		(fields_autoplaced yes)
-		(property "Reference" "#PWR019"
+		(property "Reference" "#PWR03"
 			(at 135.89 81.28 0)
 			(effects
@@
 		)
 		(instances
-			(project ""
-				(path "/b6a8d14b-6e32-4628-bf0c-2046877d1cfa/38184d55-d9c0-48fd-bb15-ff1076c43a13"
-					(reference "#PWR019")
+			(project "IMU_V100"
+				(path "/b6a8d14b-6e32-4628-bf0c-2046877d1cfa/205555cc-3b86-4915-975e-3a7e3eed6661/33aef508-2230-418a-a3ff-3a2fec798c19"
+					(reference "#PWR03")
 					(unit 1)
 				)
@@
 		(dnp no)
 		(fields_autoplaced yes)
-		(property "Reference" "#PWR018"
+		(property "Reference" "#PWR04"
 			(at 135.89 119.38 0)
 			(effects
@@
 		)
 		(instances
-			(project ""
-				(path "/b6a8d14b-6e32-4628-bf0c-2046877d1cfa/38184d55-d9c0-48fd-bb15-ff1076c43a13"
-					(reference "#PWR018")
+			(project "IMU_V100"
+				(path "/b6a8d14b-6e32-4628-bf0c-2046877d1cfa/205555cc-3b86-4915-975e-3a7e3eed6661/33aef508-2230-418a-a3ff-3a2fec798c19"
+					(reference "#PWR04")
 					(unit 1)
 				)
@@
 		(dnp no)
 		(fields_autoplaced yes)
-		(property "Reference" "#PWR020"
+		(property "Reference" "#PWR01"
 			(at 123.19 81.28 0)
 			(effects
@@
 		(instances
 			(project "IMU_V100"
-				(path "/b6a8d14b-6e32-4628-bf0c-2046877d1cfa/38184d55-d9c0-48fd-bb15-ff1076c43a13"
-					(reference "#PWR020")
+				(path "/b6a8d14b-6e32-4628-bf0c-2046877d1cfa/205555cc-3b86-4915-975e-3a7e3eed6661/33aef508-2230-418a-a3ff-3a2fec798c19"
+					(reference "#PWR01")
 					(unit 1)
 				)
@@
 		(on_board yes)
 		(dnp no)
-		(property "Reference" "U4"
+		(property "Reference" "U1"
 			(at 153.67 95.2499 0)
 			(effects
@@
 		)
 		(instances
-			(project ""
-				(path "/b6a8d14b-6e32-4628-bf0c-2046877d1cfa/38184d55-d9c0-48fd-bb15-ff1076c43a13"
-					(reference "U4")
+			(project "IMU_V100"
+				(path "/b6a8d14b-6e32-4628-bf0c-2046877d1cfa/205555cc-3b86-4915-975e-3a7e3eed6661/33aef508-2230-418a-a3ff-3a2fec798c19"
+					(reference "U1")
 					(unit 1)
 				)
@@
 		(dnp no)
 		(fields_autoplaced yes)
-		(property "Reference" "#PWR021"
+		(property "Reference" "#PWR02"
 			(at 123.19 119.38 0)
 			(effects
@@
 		(instances
 			(project "IMU_V100"
-				(path "/b6a8d14b-6e32-4628-bf0c-2046877d1cfa/38184d55-d9c0-48fd-bb15-ff1076c43a13"
-					(reference "#PWR021")
+				(path "/b6a8d14b-6e32-4628-bf0c-2046877d1cfa/205555cc-3b86-4915-975e-3a7e3eed6661/33aef508-2230-418a-a3ff-3a2fec798c19"
+					(reference "#PWR02")
 					(unit 1)
 				)
@@
 		(dnp no)
 		(fields_autoplaced yes)
-		(property "Reference" "C14"
+		(property "Reference" "C2"
 			(at 139.7 95.2499 0)
 			(effects
@@
 		)
 		(instances
-			(project ""
-				(path "/b6a8d14b-6e32-4628-bf0c-2046877d1cfa/38184d55-d9c0-48fd-bb15-ff1076c43a13"
-					(reference "C14")
-					(unit 1)
-				)
+			(project "IMU_V100"
+				(path "/b6a8d14b-6e32-4628-bf0c-2046877d1cfa/205555cc-3b86-4915-975e-3a7e3eed6661/33aef508-2230-418a-a3ff-3a2fec798c19"
+					(reference "C2")
+					(unit 1)
+				)
