File: PCB/DEBUG.kicad_sch (KiCad schematic)
At the start: 10 parts, among them J4 Conn_ARM_SWD_TagConnect_TC2030

Commit message: Updated PCB.
Parts:
- renumbered C17 to C3, C18 to C4, D4 to D1, D7 to D2, D6 to D3, D5 to D4, J4 to J2, R15 to R1, R16 to R2, R17 to R3
Changed lines of the file:
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@@
 		(on_board yes)
 		(dnp no)
-		(property "Reference" "D5"
+		(property "Reference" "D4"
 			(at 197.612 114.808 0)
 			(effects
@@
 		)
 		(instances
-			(project ""
-				(path "/b6a8d14b-6e32-4628-bf0c-2046877d1cfa/bd9088cb-f15a-411d-bc5c-97f5b7b74aa4"
-					(reference "D5")
+			(project "IMU_V100"
+				(path "/b6a8d14b-6e32-4628-bf0c-2046877d1cfa/205555cc-3b86-4915-975e-3a7e3eed6661/5b76202c-354d-4f3a-a8c9-7a4a418bf80a"
+					(reference "D4")
 					(unit 1)
 				)
@@
 		(dnp no)
 		(fields_autoplaced yes)
-		(property "Reference" "#PWR032"
+		(property "Reference" "#PWR09"
 			(at 182.88 134.62 0)
 			(effects
@@
 		(instances
 			(project "IMU_V100"
-				(path "/b6a8d14b-6e32-4628-bf0c-2046877d1cfa/bd9088cb-f15a-411d-bc5c-97f5b7b74aa4"
-					(reference "#PWR032")
+				(path "/b6a8d14b-6e32-4628-bf0c-2046877d1cfa/205555cc-3b86-4915-975e-3a7e3eed6661/5b76202c-354d-4f3a-a8c9-7a4a418bf80a"
+					(reference "#PWR09")
 					(unit 1)
 				)
@@
 		(dnp no)
 		(fields_autoplaced yes)
-		(property "Reference" "C17"
+		(property "Reference" "C3"
 			(at 166.37 69.8499 0)
 			(effects
@@
 		)
 		(instances
-			(project ""
-				(path "/b6a8d14b-6e32-4628-bf0c-2046877d1cfa/bd9088cb-f15a-411d-bc5c-97f5b7b74aa4"
-					(reference "C17")
+			(project "IMU_V100"
+				(path "/b6a8d14b-6e32-4628-bf0c-2046877d1cfa/205555cc-3b86-4915-975e-3a7e3eed6661/5b76202c-354d-4f3a-a8c9-7a4a418bf80a"
+					(reference "C3")
 					(unit 1)
 				)
@@
 		(on_board yes)
 		(dnp no)
-		(property "Reference" "R15"
+		(property "Reference" "R1"
 			(at 164.338 106.934 90)
 			(effects
@@
 		)
 		(instances
-			(project ""
-				(path "/b6a8d14b-6e32-4628-bf0c-2046877d1cfa/bd9088cb-f15a-411d-bc5c-97f5b7b74aa4"
-					(reference "R15")
+			(project "IMU_V100"
+				(path "/b6a8d14b-6e32-4628-bf0c-2046877d1cfa/205555cc-3b86-4915-975e-3a7e3eed6661/5b76202c-354d-4f3a-a8c9-7a4a418bf80a"
+					(reference "R1")
 					(unit 1)
 				)
@@
 		(dnp no)
 		(fields_autoplaced yes)
-		(property "Reference" "#PWR031"
+		(property "Reference" "#PWR010"
 			(at 189.23 134.62 0)
 			(effects
@@
 		(instances
 			(project "IMU_V100"
-				(path "/b6a8d14b-6e32-4628-bf0c-2046877d1cfa/bd9088cb-f15a-411d-bc5c-97f5b7b74aa4"
-					(reference "#PWR031")
+				(path "/b6a8d14b-6e32-4628-bf0c-2046877d1cfa/205555cc-3b86-4915-975e-3a7e3eed6661/5b76202c-354d-4f3a-a8c9-7a4a418bf80a"
+					(reference "#PWR010")
 					(unit 1)
 				)
@@
 		(dnp no)
 		(fields_autoplaced yes)
-		(property "Reference" "C18"
+		(property "Reference" "C4"
 			(at 179.07 69.8499 0)
 			(effects
@@
 		(instances
 			(project "IMU_V100"
-				(path "/b6a8d14b-6e32-4628-bf0c-2046877d1cfa/bd9088cb-f15a-411d-bc5c-97f5b7b74aa4"
-					(reference "C18")
+				(path "/b6a8d14b-6e32-4628-bf0c-2046877d1cfa/205555cc-3b86-4915-975e-3a7e3eed6661/5b76202c-354d-4f3a-a8c9-7a4a418bf80a"
+					(reference "C4")
 					(unit 1)
 				)
@@
 		(dnp no)
 		(fields_autoplaced yes)
-		(property "Reference" "#PWR029"
+		(property "Reference" "#PWR07"
 			(at 139.7 123.19 0)
 			(effects
@@
 		(instances
 			(project "IMU_V100"
-				(path "/b6a8d14b-6e32-4628-bf0c-2046877d1cfa/bd9088cb-f15a-411d-bc5c-97f5b7b74aa4"
-					(reference "#PWR029")
+				(path "/b6a8d14b-6e32-4628-bf0c-2046877d1cfa/205555cc-3b86-4915-975e-3a7e3eed6661/5b76202c-354d-4f3a-a8c9-7a4a418bf80a"
+					(reference "#PWR07")
 					(unit 1)
 				)
@@
 		(dnp no)
 		(fields_autoplaced yes)
-		(property "Reference" "#PWR022"
+		(property "Reference" "#PWR08"
 			(at 162.56 90.17 0)
 			(effects
@@
 		)
 		(instances
-			(project ""
-				(path "/b6a8d14b-6e32-4628-bf0c-2046877d1cfa/bd9088cb-f15a-411d-bc5c-97f5b7b74aa4"
-					(reference "#PWR022")
+			(project "IMU_V100"
+				(path "/b6a8d14b-6e32-4628-bf0c-2046877d1cfa/205555cc-3b86-4915-975e-3a7e3eed6661/5b76202c-354d-4f3a-a8c9-7a4a418bf80a"
+					(reference "#PWR08")
 					(unit 1)
 				)
@@
 		(dnp no)
 		(fields_autoplaced yes)
-		(property "Reference" "D4"
+		(property "Reference" "D1"
 			(at 148.59 69.8499 90)
 			(effects
@@
 		)
 		(instances
-			(project ""
-				(path "/b6a8d14b-6e32-4628-bf0c-2046877d1cfa/bd9088cb-f15a-411d-bc5c-97f5b7b74aa4"
-					(reference "D4")
+			(project "IMU_V100"
+				(path "/b6a8d14b-6e32-4628-bf0c-2046877d1cfa/205555cc-3b86-4915-975e-3a7e3eed6661/5b76202c-354d-4f3a-a8c9-7a4a418bf80a"
+					(reference "D1")
 					(unit 1)
 				)
@@
 		(on_board yes)
 		(dnp no)
-		(property "Reference" "D7"
+		(property "Reference" "D2"
 			(at 184.912 114.808 0)
 			(effects
@@
 		(instances
 			(project "IMU_V100"
-				(path "/b6a8d14b-6e32-4628-bf0c-2046877d1cfa/bd9088cb-f15a-411d-bc5c-97f5b7b74aa4"
-					(reference "D7")
+				(path "/b6a8d14b-6e32-4628-bf0c-2046877d1cfa/205555cc-3b86-4915-975e-3a7e3eed6661/5b76202c-354d-4f3a-a8c9-7a4a418bf80a"
+					(reference "D2")
 					(unit 1)
 				)
@@
 		(on_board yes)
 		(dnp no)
-		(property "Reference" "R17"
+		(property "Reference" "R3"
 			(at 191.008 101.854 90)
 			(effects
@@
 		(instances
 			(project "IMU_V100"
-				(path "/b6a8d14b-6e32-4628-bf0c-2046877d1cfa/bd9088cb-f15a-411d-bc5c-97f5b7b74aa4"
-					(reference "R17")
+				(path "/b6a8d14b-6e32-4628-bf0c-2046877d1cfa/205555cc-3b86-4915-975e-3a7e3eed6661/5b76202c-354d-4f3a-a8c9-7a4a418bf80a"
+					(reference "R3")
 					(unit 1)
 				)
@@
 		(on_board yes)
 		(dnp no)
-		(property "Reference" "D6"
+		(property "Reference" "D3"
 			(at 191.262 114.808 0)
 			(effects
@@
 		(instances
 			(project "IMU_V100"
-				(path "/b6a8d14b-6e32-4628-bf0c-2046877d1cfa/bd9088cb-f15a-411d-bc5c-97f5b7b74aa4"
-					(reference "D6")
+				(path "/b6a8d14b-6e32-4628-bf0c-2046877d1cfa/205555cc-3b86-4915-975e-3a7e3eed6661/5b76202c-354d-4f3a-a8c9-7a4a418bf80a"
+					(reference "D3")
 					(unit 1)
 				)
@@
 		(dnp no)
 		(fields_autoplaced yes)
-		(property "Reference" "#PWR030"
+		(property "Reference" "#PWR011"
 			(at 195.58 134.62 0)
 			(effects
@@
 		(instances
 			(project "IMU_V100"
-				(path "/b6a8d14b-6e32-4628-bf0c-2046877d1cfa/bd9088cb-f15a-411d-bc5c-97f5b7b74aa4"
-					(reference "#PWR030")
+				(path "/b6a8d14b-6e32-4628-bf0c-2046877d1cfa/205555cc-3b86-4915-975e-3a7e3eed6661/5b76202c-354d-4f3a-a8c9-7a4a418bf80a"
+					(reference "#PWR011")
 					(unit 1)
 				)
@@
 		(on_board yes)
 		(dnp no)
-		(property "Reference" "R16"
+		(property "Reference" "R2"
 			(at 177.038 104.394 90)
 			(effects
@@
 		(instances
 			(project "IMU_V100"
-				(path "/b6a8d14b-6e32-4628-bf0c-2046877d1cfa/bd9088cb-f15a-411d-bc5c-97f5b7b74aa4"
-					(reference "R16")
+				(path "/b6a8d14b-6e32-4628-bf0c-2046877d1cfa/205555cc-3b86-4915-975e-3a7e3eed6661/5b76202c-354d-4f3a-a8c9-7a4a418bf80a"
+					(reference "R2")
 					(unit 1)
 				)
@@
 		(dnp no)
 		(fields_autoplaced yes)
-		(property "Reference" "J4"
+		(property "Reference" "J2"
 			(at 135.89 101.5999 0)
 			(effects
@@
 		)
 		(instances
-			(project ""
-				(path "/b6a8d14b-6e32-4628-bf0c-2046877d1cfa/bd9088cb-f15a-411d-bc5c-97f5b7b74aa4"
-					(reference "J4")
-					(unit 1)
-				)
+			(project "IMU_V100"
+				(path "/b6a8d14b-6e32-4628-bf0c-2046877d1cfa/205555cc-3b86-4915-975e-3a7e3eed6661/5b76202c-354d-4f3a-a8c9-7a4a418bf80a"
+					(reference "J2")
+					(unit 1)
+				)
