File: PCB/DEBUG.kicad_sch (KiCad schematic)
At the start: 10 parts, among them J2 Conn_ARM_SWD_TagConnect_TC2030

Commit message: Updated PCB
Parts:
- renumbered C3 to C5, C4 to C6, R1 to R3, R2 to R4, R3 to R5
Changed lines of the file:
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@@
 		(dnp no)
 		(fields_autoplaced yes)
-		(property "Reference" "#PWR09"
+		(property "Reference" "#PWR012"
 			(at 182.88 134.62 0)
 			(effects
@@
 			(project "IMU_V100"
 				(path "/b6a8d14b-6e32-4628-bf0c-2046877d1cfa/205555cc-3b86-4915-975e-3a7e3eed6661/5b76202c-354d-4f3a-a8c9-7a4a418bf80a"
-					(reference "#PWR09")
+					(reference "#PWR012")
 					(unit 1)
 				)
@@
 		(dnp no)
 		(fields_autoplaced yes)
-		(property "Reference" "C3"
+		(property "Reference" "C5"
 			(at 166.37 69.8499 0)
 			(effects
@@
 			(project "IMU_V100"
 				(path "/b6a8d14b-6e32-4628-bf0c-2046877d1cfa/205555cc-3b86-4915-975e-3a7e3eed6661/5b76202c-354d-4f3a-a8c9-7a4a418bf80a"
-					(reference "C3")
+					(reference "C5")
 					(unit 1)
 				)
@@
 		(on_board yes)
 		(dnp no)
-		(property "Reference" "R1"
+		(property "Reference" "R3"
 			(at 164.338 106.934 90)
 			(effects
@@
 			(project "IMU_V100"
 				(path "/b6a8d14b-6e32-4628-bf0c-2046877d1cfa/205555cc-3b86-4915-975e-3a7e3eed6661/5b76202c-354d-4f3a-a8c9-7a4a418bf80a"
-					(reference "R1")
+					(reference "R3")
 					(unit 1)
 				)
@@
 		(dnp no)
 		(fields_autoplaced yes)
-		(property "Reference" "#PWR010"
+		(property "Reference" "#PWR013"
 			(at 189.23 134.62 0)
 			(effects
@@
 			(project "IMU_V100"
 				(path "/b6a8d14b-6e32-4628-bf0c-2046877d1cfa/205555cc-3b86-4915-975e-3a7e3eed6661/5b76202c-354d-4f3a-a8c9-7a4a418bf80a"
-					(reference "#PWR010")
+					(reference "#PWR013")
 					(unit 1)
 				)
@@
 		(dnp no)
 		(fields_autoplaced yes)
-		(property "Reference" "C4"
+		(property "Reference" "C6"
 			(at 179.07 69.8499 0)
 			(effects
@@
 			(project "IMU_V100"
 				(path "/b6a8d14b-6e32-4628-bf0c-2046877d1cfa/205555cc-3b86-4915-975e-3a7e3eed6661/5b76202c-354d-4f3a-a8c9-7a4a418bf80a"
-					(reference "C4")
+					(reference "C6")
 					(unit 1)
 				)
@@
 		(dnp no)
 		(fields_autoplaced yes)
-		(property "Reference" "#PWR07"
+		(property "Reference" "#PWR010"
 			(at 139.7 123.19 0)
 			(effects
@@
 			(project "IMU_V100"
 				(path "/b6a8d14b-6e32-4628-bf0c-2046877d1cfa/205555cc-3b86-4915-975e-3a7e3eed6661/5b76202c-354d-4f3a-a8c9-7a4a418bf80a"
-					(reference "#PWR07")
+					(reference "#PWR010")
 					(unit 1)
 				)
@@
 		(dnp no)
 		(fields_autoplaced yes)
-		(property "Reference" "#PWR08"
+		(property "Reference" "#PWR011"
 			(at 162.56 90.17 0)
 			(effects
@@
 			(project "IMU_V100"
 				(path "/b6a8d14b-6e32-4628-bf0c-2046877d1cfa/205555cc-3b86-4915-975e-3a7e3eed6661/5b76202c-354d-4f3a-a8c9-7a4a418bf80a"
-					(reference "#PWR08")
+					(reference "#PWR011")
 					(unit 1)
 				)
@@
 		(on_board yes)
 		(dnp no)
-		(property "Reference" "R3"
+		(property "Reference" "R5"
 			(at 191.008 101.854 90)
 			(effects
@@
 			(project "IMU_V100"
 				(path "/b6a8d14b-6e32-4628-bf0c-2046877d1cfa/205555cc-3b86-4915-975e-3a7e3eed6661/5b76202c-354d-4f3a-a8c9-7a4a418bf80a"
-					(reference "R3")
+					(reference "R5")
 					(unit 1)
 				)
@@
 		(dnp no)
 		(fields_autoplaced yes)
-		(property "Reference" "#PWR011"
+		(property "Reference" "#PWR014"
 			(at 195.58 134.62 0)
 			(effects
@@
 			(project "IMU_V100"
 				(path "/b6a8d14b-6e32-4628-bf0c-2046877d1cfa/205555cc-3b86-4915-975e-3a7e3eed6661/5b76202c-354d-4f3a-a8c9-7a4a418bf80a"
-					(reference "#PWR011")
+					(reference "#PWR014")
 					(unit 1)
 				)
@@
 		(on_board yes)
 		(dnp no)
-		(property "Reference" "R2"
+		(property "Reference" "R4"
 			(at 177.038 104.394 90)
 			(effects
@@
 			(project "IMU_V100"
 				(path "/b6a8d14b-6e32-4628-bf0c-2046877d1cfa/205555cc-3b86-4915-975e-3a7e3eed6661/5b76202c-354d-4f3a-a8c9-7a4a418bf80a"
-					(reference "R2")
-					(unit 1)
-				)
+					(reference "R4")
+					(unit 1)
+				)
