File: PCB/GPS.kicad_sch (KiCad schematic)
At the start: 23 parts, among them IC1 LC76GABMD, J2 Conn_01x04

Commit message: Updated PCB.
Parts:
- renumbered C12 to C10, C9 to C11, C10 to C12, C11 to C7, C7 to C9, D1 to D5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
