File: PCB/GPS.kicad_sch (KiCad schematic)
At the start: 23 parts, among them IC1 LC76GABMD, J3 Conn_01x04

Commit message: Updated PCB
Parts:
- C10, C11, C12, C13, C5, C6, C7, C8, C9: footprint (none) -> Capacitor_SMD:C_0402_1005Metric_Pad0.74x0.62mm_HandSolder
- R10, R11, R4, R5, R6, R7, R8, R9: footprint (none) -> Resistor_SMD:R_0402_1005Metric
Changed lines of the file:
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@@
 			)
 		)
-		(property "Footprint" ""
+		(property "Footprint" "Capacitor_SMD:C_0402_1005Metric_Pad0.74x0.62mm_HandSolder"
 			(at 67.31 60.96 0)
 			(effects
@@
 			)
 		)
-		(property "Footprint" ""
+		(property "Footprint" "Resistor_SMD:R_0402_1005Metric"
 			(at 224.79 64.77 0)
 			(effects
@@
 			)
 		)
-		(property "Footprint" ""
+		(property "Footprint" "Capacitor_SMD:C_0402_1005Metric_Pad0.74x0.62mm_HandSolder"
 			(at 55.88 90.17 0)
 			(effects
@@
 			)
 		)
-		(property "Footprint" ""
+		(property "Footprint" "Resistor_SMD:R_0402_1005Metric"
 			(at 220.98 64.77 0)
 			(effects
@@
 			)
 		)
-		(property "Footprint" ""
+		(property "Footprint" "Capacitor_SMD:C_0402_1005Metric_Pad0.74x0.62mm_HandSolder"
 			(at 68.58 90.17 0)
 			(effects
@@
 			)
 		)
-		(property "Footprint" ""
+		(property "Footprint" "Resistor_SMD:R_0402_1005Metric"
 			(at 210.82 81.28 0)
 			(effects
@@
 			)
 		)
-		(property "Footprint" ""
+		(property "Footprint" "Capacitor_SMD:C_0402_1005Metric_Pad0.74x0.62mm_HandSolder"
 			(at 44.45 90.17 0)
 			(effects
@@
 			)
 		)
-		(property "Footprint" ""
+		(property "Footprint" "Capacitor_SMD:C_0402_1005Metric_Pad0.74x0.62mm_HandSolder"
 			(at 93.98 149.86 0)
 			(effects
@@
 			)
 		)
-		(property "Footprint" ""
+		(property "Footprint" "Capacitor_SMD:C_0402_1005Metric_Pad0.74x0.62mm_HandSolder"
 			(at 78.74 60.96 0)
 			(effects
@@
 			)
 		)
-		(property "Footprint" ""
+		(property "Footprint" "Resistor_SMD:R_0402_1005Metric"
 			(at 252.73 87.63 0)
 			(effects
@@
 			)
 		)
-		(property "Footprint" ""
+		(property "Footprint" "Capacitor_SMD:C_0402_1005Metric_Pad0.74x0.62mm_HandSolder"
 			(at 91.44 60.96 0)
 			(effects
@@
 			)
 		)
-		(property "Footprint" ""
+		(property "Footprint" "Resistor_SMD:R_0402_1005Metric"
 			(at 83.82 135.89 0)
 			(effects
@@
 			)
 		)
-		(property "Footprint" ""
+		(property "Footprint" "Resistor_SMD:R_0402_1005Metric"
 			(at 210.82 86.36 0)
 			(effects
@@
 			)
 		)
-		(property "Footprint" ""
+		(property "Footprint" "Capacitor_SMD:C_0402_1005Metric_Pad0.74x0.62mm_HandSolder"
 			(at 64.77 135.89 0)
 			(effects
@@
 			)
 		)
-		(property "Footprint" ""
+		(property "Footprint" "Capacitor_SMD:C_0402_1005Metric_Pad0.74x0.62mm_HandSolder"
 			(at 74.93 149.86 0)
 			(effects
@@
 			)
 		)
-		(property "Footprint" ""
+		(property "Footprint" "Resistor_SMD:R_0402_1005Metric"
 			(at 124.46 100.33 0)
 			(effects
@@
 			)
 		)
-		(property "Footprint" ""
+		(property "Footprint" "Resistor_SMD:R_0402_1005Metric"
 			(at 99.06 123.19 0)
 			(effects

Commit message: Updated PCB
Parts:
- renumbered C8 to C10, C9 to C11, C10 to C12, C11 to C13, C12 to C14, C13 to C15, C5 to C7, C6 to C8, C7 to C9, R8 to R10, R9 to R11, R10 to R12, R11 to R13, R4 to R6, R5 to R7, R6 to R8, R7 to R9
Changed lines of the file:
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@@
 		(dnp no)
 		(fields_autoplaced yes)
-		(property "Reference" "C8"
+		(property "Reference" "C10"
 			(at 71.12 59.6899 0)
 			(effects
@@
 			(project "IMU_V100"
 				(path "/b6a8d14b-6e32-4628-bf0c-2046877d1cfa/205555cc-3b86-4915-975e-3a7e3eed6661/ea59acea-8322-4969-ac03-70a626785633"
-					(reference "C8")
+					(reference "C10")
 					(unit 1)
 				)
@@
 		(dnp no)
 		(fields_autoplaced yes)
-		(property "Reference" "#PWR017"
+		(property "Reference" "#PWR020"
 			(at 134.62 109.22 0)
 			(effects
@@
 			(project "IMU_V100"
 				(path "/b6a8d14b-6e32-4628-bf0c-2046877d1cfa/205555cc-3b86-4915-975e-3a7e3eed6661/ea59acea-8322-4969-ac03-70a626785633"
-					(reference "#PWR017")
+					(reference "#PWR020")
 					(unit 1)
 				)
@@
 		(dnp no)
 		(fields_autoplaced yes)
-		(property "Reference" "#PWR012"
+		(property "Reference" "#PWR015"
 			(at 34.29 76.2 0)
 			(effects
@@
 			(project "IMU_V100"
 				(path "/b6a8d14b-6e32-4628-bf0c-2046877d1cfa/205555cc-3b86-4915-975e-3a7e3eed6661/ea59acea-8322-4969-ac03-70a626785633"
-					(reference "#PWR012")
+					(reference "#PWR015")
 					(unit 1)
 				)
@@
 		(on_board yes)
 		(dnp no)
-		(property "Reference" "R10"
+		(property "Reference" "R12"
 			(at 226.06 60.706 90)
 			(effects
@@
 			(project "IMU_V100"
 				(path "/b6a8d14b-6e32-4628-bf0c-2046877d1cfa/205555cc-3b86-4915-975e-3a7e3eed6661/ea59acea-8322-4969-ac03-70a626785633"
-					(reference "R10")
+					(reference "R12")
 					(unit 1)
 				)
@@
 		(dnp no)
 		(fields_autoplaced yes)
-		(property "Reference" "#PWR020"
+		(property "Reference" "#PWR023"
 			(at 209.55 127 0)
 			(effects
@@
 			(project "IMU_V100"
 				(path "/b6a8d14b-6e32-4628-bf0c-2046877d1cfa/205555cc-3b86-4915-975e-3a7e3eed6661/ea59acea-8322-4969-ac03-70a626785633"
-					(reference "#PWR020")
+					(reference "#PWR023")
 					(unit 1)
 				)
@@
 		(dnp no)
 		(fields_autoplaced yes)
-		(property "Reference" "C6"
+		(property "Reference" "C8"
 			(at 59.69 88.8999 0)
 			(effects
@@
 			(project "IMU_V100"
 				(path "/b6a8d14b-6e32-4628-bf0c-2046877d1cfa/205555cc-3b86-4915-975e-3a7e3eed6661/ea59acea-8322-4969-ac03-70a626785633"
-					(reference "C6")
+					(reference "C8")
 					(unit 1)
 				)
@@
 		(on_board yes)
 		(dnp no)
-		(property "Reference" "R9"
+		(property "Reference" "R11"
 			(at 222.25 60.706 90)
 			(effects
@@
 			(project "IMU_V100"
 				(path "/b6a8d14b-6e32-4628-bf0c-2046877d1cfa/205555cc-3b86-4915-975e-3a7e3eed6661/ea59acea-8322-4969-ac03-70a626785633"
-					(reference "R9")
+					(reference "R11")
 					(unit 1)
 				)
@@
 		(dnp no)
 		(fields_autoplaced yes)
-		(property "Reference" "C9"
+		(property "Reference" "C11"
 			(at 72.39 88.8999 0)
 			(effects
@@
 			(project "IMU_V100"
 				(path "/b6a8d14b-6e32-4628-bf0c-2046877d1cfa/205555cc-3b86-4915-975e-3a7e3eed6661/ea59acea-8322-4969-ac03-70a626785633"
-					(reference "C9")
+					(reference "C11")
 					(unit 1)
 				)
@@
 		(on_board yes)
 		(dnp no)
-		(property "Reference" "R7"
+		(property "Reference" "R9"
 			(at 212.09 78.74 90)
 			(effects
@@
 			(project "IMU_V100"
 				(path "/b6a8d14b-6e32-4628-bf0c-2046877d1cfa/205555cc-3b86-4915-975e-3a7e3eed6661/ea59acea-8322-4969-ac03-70a626785633"
-					(reference "R7")
+					(reference "R9")
 					(unit 1)
 				)
@@
 		(dnp no)
 		(fields_autoplaced yes)
-		(property "Reference" "C5"
+		(property "Reference" "C7"
 			(at 48.26 88.8999 0)
 			(effects
@@
 			(project "IMU_V100"
 				(path "/b6a8d14b-6e32-4628-bf0c-2046877d1cfa/205555cc-3b86-4915-975e-3a7e3eed6661/ea59acea-8322-4969-ac03-70a626785633"
-					(reference "C5")
+					(reference "C7")
 					(unit 1)
 				)
@@
 		(dnp no)
 		(fields_autoplaced yes)
-		(property "Reference" "#PWR019"
+		(property "Reference" "#PWR022"
 			(at 153.67 128.27 0)
 			(effects
@@
 			(project "IMU_V100"
 				(path "/b6a8d14b-6e32-4628-bf0c-2046877d1cfa/205555cc-3b86-4915-975e-3a7e3eed6661/ea59acea-8322-4969-ac03-70a626785633"
-					(reference "#PWR019")
+					(reference "#PWR022")
 					(unit 1)
 				)
@@
 		(dnp no)
 		(fields_autoplaced yes)
-		(property "Reference" "C13"
+		(property "Reference" "C15"
 			(at 97.79 148.5899 0)
 			(effects
@@
 			(project "IMU_V100"
 				(path "/b6a8d14b-6e32-4628-bf0c-2046877d1cfa/205555cc-3b86-4915-975e-3a7e3eed6661/ea59acea-8322-4969-ac03-70a626785633"
-					(reference "C13")
+					(reference "C15")
 					(unit 1)
 				)
@@
 		(dnp no)
 		(fields_autoplaced yes)
-		(property "Reference" "C11"
+		(property "Reference" "C13"
 			(at 82.55 59.6899 0)
 			(effects
@@
 			(project "IMU_V100"
 				(path "/b6a8d14b-6e32-4628-bf0c-2046877d1cfa/205555cc-3b86-4915-975e-3a7e3eed6661/ea59acea-8322-4969-ac03-70a626785633"
-					(reference "C11")
+					(reference "C13")
 					(unit 1)
 				)
@@
 		(dnp no)
 		(fields_autoplaced yes)
-		(property "Reference" "#PWR013"
+		(property "Reference" "#PWR016"
 			(at 39.37 149.86 0)
 			(effects
@@
 			(project "IMU_V100"
 				(path "/b6a8d14b-6e32-4628-bf0c-2046877d1cfa/205555cc-3b86-4915-975e-3a7e3eed6661/ea59acea-8322-4969-ac03-70a626785633"
-					(reference "#PWR013")
+					(reference "#PWR016")
 					(unit 1)
 				)
@@
 		(dnp no)
 		(fields_autoplaced yes)
-		(property "Reference" "R11"
+		(property "Reference" "R13"
 			(at 255.27 87.6299 0)
 			(effects
@@
 			(project "IMU_V100"
 				(path "/b6a8d14b-6e32-4628-bf0c-2046877d1cfa/205555cc-3b86-4915-975e-3a7e3eed6661/ea59acea-8322-4969-ac03-70a626785633"
-					(reference "R11")
+					(reference "R13")
 					(unit 1)
 				)
@@
 		(dnp no)
 		(fields_autoplaced yes)
-		(property "Reference" "#PWR014"
+		(property "Reference" "#PWR017"
 			(at 44.45 109.22 0)
 			(effects
@@
 			(project "IMU_V100"
 				(path "/b6a8d14b-6e32-4628-bf0c-2046877d1cfa/205555cc-3b86-4915-975e-3a7e3eed6661/ea59acea-8322-4969-ac03-70a626785633"
-					(reference "#PWR014")
+					(reference "#PWR017")
 					(unit 1)
 				)
@@
 		(dnp no)
 		(fields_autoplaced yes)
-		(property "Reference" "C12"
+		(property "Reference" "C14"
 			(at 95.25 59.6899 0)
 			(effects
@@
 			(project "IMU_V100"
 				(path "/b6a8d14b-6e32-4628-bf0c-2046877d1cfa/205555cc-3b86-4915-975e-3a7e3eed6661/ea59acea-8322-4969-ac03-70a626785633"
-					(reference "C12")
+					(reference "C14")
 					(unit 1)
 				)
@@
 		(dnp no)
 		(fields_autoplaced yes)
-		(property "Reference" "R4"
+		(property "Reference" "R6"
 			(at 83.82 132.08 90)
 			(effects
@@
 			(project "IMU_V100"
 				(path "/b6a8d14b-6e32-4628-bf0c-2046877d1cfa/205555cc-3b86-4915-975e-3a7e3eed6661/ea59acea-8322-4969-ac03-70a626785633"
-					(reference "R4")
+					(reference "R6")
 					(unit 1)
 				)
@@
 		(on_board yes)
 		(dnp no)
-		(property "Reference" "R8"
+		(property "Reference" "R10"
 			(at 217.424 85.09 90)
 			(effects
@@
 			(project "IMU_V100"
 				(path "/b6a8d14b-6e32-4628-bf0c-2046877d1cfa/205555cc-3b86-4915-975e-3a7e3eed6661/ea59acea-8322-4969-ac03-70a626785633"
-					(reference "R8")
+					(reference "R10")
 					(unit 1)
 				)
@@
 		(dnp no)
 		(fields_autoplaced yes)
-		(property "Reference" "C7"
+		(property "Reference" "C9"
 			(at 64.77 129.54 90)
 			(effects
@@
 			(project "IMU_V100"
 				(path "/b6a8d14b-6e32-4628-bf0c-2046877d1cfa/205555cc-3b86-4915-975e-3a7e3eed6661/ea59acea-8322-4969-ac03-70a626785633"
-					(reference "C7")
+					(reference "C9")
 					(unit 1)
 				)
@@
 		(dnp no)
 		(fields_autoplaced yes)
-		(property "Reference" "#PWR015"
+		(property "Reference" "#PWR018"
 			(at 49.53 130.81 0)
 			(effects
@@
 			(project "IMU_V100"
 				(path "/b6a8d14b-6e32-4628-bf0c-2046877d1cfa/205555cc-3b86-4915-975e-3a7e3eed6661/ea59acea-8322-4969-ac03-70a626785633"
-					(reference "#PWR015")
+					(reference "#PWR018")
 					(unit 1)
 				)
@@
 		(dnp no)
 		(fields_autoplaced yes)
-		(property "Reference" "#PWR016"
+		(property "Reference" "#PWR019"
 			(at 85.09 172.72 0)
 			(effects
@@
 			(project "IMU_V100"
 				(path "/b6a8d14b-6e32-4628-bf0c-2046877d1cfa/205555cc-3b86-4915-975e-3a7e3eed6661/ea59acea-8322-4969-ac03-70a626785633"
-					(reference "#PWR016")
+					(reference "#PWR019")
 					(unit 1)
 				)
@@
 		(dnp no)
 		(fields_autoplaced yes)
-		(property "Reference" "C10"
+		(property "Reference" "C12"
 			(at 78.74 148.5899 0)
 			(effects
@@
 			(project "IMU_V100"
 				(path "/b6a8d14b-6e32-4628-bf0c-2046877d1cfa/205555cc-3b86-4915-975e-3a7e3eed6661/ea59acea-8322-4969-ac03-70a626785633"
-					(reference "C10")
+					(reference "C12")
 					(unit 1)
 				)
@@
 		(on_board yes)
 		(dnp no)
-		(property "Reference" "R6"
+		(property "Reference" "R8"
 			(at 131.064 99.06 90)
 			(effects
@@
 			(project "IMU_V100"
 				(path "/b6a8d14b-6e32-4628-bf0c-2046877d1cfa/205555cc-3b86-4915-975e-3a7e3eed6661/ea59acea-8322-4969-ac03-70a626785633"
-					(reference "R6")
+					(reference "R8")
 					(unit 1)
 				)
@@
 		(dnp no)
 		(fields_autoplaced yes)
-		(property "Reference" "#PWR018"
+		(property "Reference" "#PWR021"
 			(at 153.67 77.47 0)
 			(effects
@@
 			(project "IMU_V100"
 				(path "/b6a8d14b-6e32-4628-bf0c-2046877d1cfa/205555cc-3b86-4915-975e-3a7e3eed6661/ea59acea-8322-4969-ac03-70a626785633"
-					(reference "#PWR018")
+					(reference "#PWR021")
 					(unit 1)
 				)
@@
 		(dnp no)
 		(fields_autoplaced yes)
-		(property "Reference" "R5"
+		(property "Reference" "R7"
 			(at 99.06 119.38 90)
 			(effects
@@
 			(project "IMU_V100"
 				(path "/b6a8d14b-6e32-4628-bf0c-2046877d1cfa/205555cc-3b86-4915-975e-3a7e3eed6661/ea59acea-8322-4969-ac03-70a626785633"
-					(reference "R5")
-					(unit 1)
-				)
+					(reference "R7")
+					(unit 1)
+				)
