File: PCB/Block_Diagram.kicad_sch (KiCad schematic)
At the start: 0 parts

Commit message: Updated PCB.
Other:
- note removed: "DEBUG"
- note removed: "I2C"
- note removed: "POWER"
- note removed: "SIGNALS"
- note removed: "SPI"
- note removed: "UART"
