File: PCB/CAN_FD.kicad_sch (KiCad schematic)
At the start: 2 parts, among them J3 Conn_01x04, U5 MCP2557FD-xMNY

Commit message: Updated PCB.
Parts:
- renumbered J3 to J1, U5 to U2
Changed lines of the file:
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@@
 		(dnp no)
 		(fields_autoplaced yes)
-		(property "Reference" "#PWR016"
+		(property "Reference" "#PWR05"
 			(at 129.54 121.92 0)
 			(effects
@@
 		)
 		(instances
-			(project ""
-				(path "/b6a8d14b-6e32-4628-bf0c-2046877d1cfa/8e7c721f-4787-45c0-877a-ccbe11a9aa6f"
-					(reference "#PWR016")
+			(project "IMU_V100"
+				(path "/b6a8d14b-6e32-4628-bf0c-2046877d1cfa/205555cc-3b86-4915-975e-3a7e3eed6661/0bf2e565-c24a-4992-bfd2-1fa1b050084a"
+					(reference "#PWR05")
 					(unit 1)
 				)
@@
 		(dnp no)
 		(fields_autoplaced yes)
-		(property "Reference" "U5"
+		(property "Reference" "U2"
 			(at 131.7341 85.09 0)
 			(effects
@@
 		)
 		(instances
-			(project ""
-				(path "/b6a8d14b-6e32-4628-bf0c-2046877d1cfa/8e7c721f-4787-45c0-877a-ccbe11a9aa6f"
-					(reference "U5")
+			(project "IMU_V100"
+				(path "/b6a8d14b-6e32-4628-bf0c-2046877d1cfa/205555cc-3b86-4915-975e-3a7e3eed6661/0bf2e565-c24a-4992-bfd2-1fa1b050084a"
+					(reference "U2")
 					(unit 1)
 				)
@@
 		(dnp no)
 		(fields_autoplaced yes)
-		(property "Reference" "J3"
+		(property "Reference" "J1"
 			(at 198.12 95.2499 0)
 			(effects
@@
 		)
 		(instances
-			(project ""
-				(path "/b6a8d14b-6e32-4628-bf0c-2046877d1cfa/8e7c721f-4787-45c0-877a-ccbe11a9aa6f"
-					(reference "J3")
+			(project "IMU_V100"
+				(path "/b6a8d14b-6e32-4628-bf0c-2046877d1cfa/205555cc-3b86-4915-975e-3a7e3eed6661/0bf2e565-c24a-4992-bfd2-1fa1b050084a"
+					(reference "J1")
 					(unit 1)
 				)
@@
 		(dnp no)
 		(fields_autoplaced yes)
-		(property "Reference" "#PWR017"
+		(property "Reference" "#PWR06"
 			(at 182.88 118.11 0)
 			(effects
@@
 		)
 		(instances
-			(project ""
-				(path "/b6a8d14b-6e32-4628-bf0c-2046877d1cfa/8e7c721f-4787-45c0-877a-ccbe11a9aa6f"
-					(reference "#PWR017")
-					(unit 1)
-				)
+			(project "IMU_V100"
+				(path "/b6a8d14b-6e32-4628-bf0c-2046877d1cfa/205555cc-3b86-4915-975e-3a7e3eed6661/0bf2e565-c24a-4992-bfd2-1fa1b050084a"
+					(reference "#PWR06")
+					(unit 1)
+				)

Commit message: Updated PCB.
Parts:
- removed J1: Conn_01x04, symbol Connector_Generic:Conn_01x04
- added C19: 0.1uF, symbol PCM_Elektuur:C
- added C20: 4700pF, symbol PCM_Elektuur:C
- added J1: 1-770969-0, Footprints:17709690, symbol IMU_V100:1-770969-0
- added R18, R19: 60R, symbol PCM_Elektuur:R
Connections:
- net GND: now also C19.1 (+), C20.1 (+), J1.4
- net VIN: now also J1.1; no longer U2.3 (VDD)
- net at U2.6 (CANL): now also J1.5, R19.1 (+)
- net at U2.7 (CANH): now also J1.2, R18.2 (-)
- new net: C20.2 (-), R18.1 (+), R19.2 (-)
- new net +3V3: C19.2 (-), U2.3 (VDD)

Commit message: Updated PCB
Connections:
- net CAN_USER1: now reaches J1.3
- net CAN_USER2: now reaches J1.6
Other:
- moved on the sheet: C20
Changed lines of the file:
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@@
 	(wire
 		(pts
-			(xy 179.07 116.84) (xy 179.07 119.38)
+			(xy 176.53 116.84) (xy 176.53 119.38)
 		)
 		(stroke
@@
 	(wire
 		(pts
+			(xy 200.66 106.68) (xy 207.01 106.68)
+		)
+		(stroke
+			(width 0)
+			(type default)
+		)
+	)
+	(wire
+		(pts
 			(xy 142.24 95.25) (xy 156.21 95.25)
 		)
@@
 	(wire
 		(pts
-			(xy 179.07 106.68) (xy 179.07 104.14)
+			(xy 176.53 106.68) (xy 176.53 104.14)
 		)
 		(stroke
@@
 	(wire
 		(pts
+			(xy 207.01 106.68) (xy 207.01 105.41)
+		)
+		(stroke
+			(width 0)
+			(type default)
+		)
+	)
+	(wire
+		(pts
 			(xy 165.1 85.09) (xy 165.1 90.17)
 		)
@@
 	(wire
 		(pts
+			(xy 198.12 83.82) (xy 207.01 83.82)
+		)
+		(stroke
+			(width 0)
+			(type default)
+		)
+	)
+	(wire
+		(pts
+			(xy 207.01 83.82) (xy 207.01 85.09)
+		)
+		(stroke
+			(width 0)
+			(type default)
+		)
+	)
+	(wire
+		(pts
 			(xy 107.95 102.87) (xy 116.84 102.87)
 		)
@@
 	(wire
 		(pts
-			(xy 165.1 104.14) (xy 179.07 104.14)
+			(xy 165.1 104.14) (xy 176.53 104.14)
 		)
 		(stroke
@@
 		)
 	)
+	(hierarchical_label "CAN_USER1"
+		(shape bidirectional)
+		(at 198.12 83.82 180)
+		(fields_autoplaced yes)
+		(effects
+			(font
+				(size 1.27 1.27)
+			)
+			(justify right)
+		)
+	)
 	(hierarchical_label "CAN_RX"
 		(shape input)
 		(at 107.95 95.25 180)
+		(fields_autoplaced yes)
+		(effects
+			(font
+				(size 1.27 1.27)
+			)
+			(justify right)
+		)
+	)
+	(hierarchical_label "CAN_USER2"
+		(shape bidirectional)
+		(at 200.66 106.68 180)
 		(fields_autoplaced yes)
 		(effects
@@
 	(symbol
 		(lib_id "PCM_Elektuur:C")
-		(at 179.07 111.76 180)
+		(at 176.53 111.76 180)
 		(unit 1)
 		(exclude_from_sim no)
@@
 		(fields_autoplaced yes)
 		(property "Reference" "C20"
-			(at 182.88 110.4899 0)
+			(at 180.34 110.4899 0)
 			(effects
 				(font
@@
 		)
 		(property "Value" "4700pF"
-			(at 182.88 113.0299 0)
+			(at 180.34 113.0299 0)
 			(effects
 				(font
@@
 		)
 		(property "Footprint" ""
-			(at 179.07 111.76 0)
+			(at 176.53 111.76 0)
 			(effects
 				(font
@@
 		)
 		(property "Datasheet" ""
-			(at 179.07 111.76 0)
+			(at 176.53 111.76 0)
 			(effects
 				(font
@@
 		)
 		(property "Description" "capacitor, non-polarized/bipolar"
-			(at 179.07 111.76 0)
+			(at 176.53 111.76 0)
 			(effects
 				(font
@@
 		)
 		(property "Indicator" "+"
-			(at 180.34 114.935 0)
+			(at 177.8 114.935 0)
 			(do_not_autoplace yes)
 			(effects
@@
 		)
 		(property "Rating" "V"
-			(at 179.705 108.585 0)
+			(at 177.165 108.585 0)
 			(effects
 				(font
@@
 	(symbol
 		(lib_id "power:GND")
-		(at 179.07 119.38 0)
+		(at 176.53 119.38 0)
 		(unit 1)
 		(exclude_from_sim no)
@@
 		(fields_autoplaced yes)
 		(property "Reference" "#PWR032"
-			(at 179.07 125.73 0)
+			(at 176.53 125.73 0)
 			(effects
 				(font
@@
 		)
 		(property "Value" "GND"
-			(at 179.07 124.46 0)
+			(at 176.53 124.46 0)
 			(effects
 				(font
@@
 		)
 		(property "Footprint" ""
-			(at 179.07 119.38 0)
+			(at 176.53 119.38 0)
 			(effects
 				(font
@@
 		)
 		(property "Datasheet" ""
-			(at 179.07 119.38 0)
+			(at 176.53 119.38 0)
 			(effects
 				(font
@@
 		)
 		(property "Description" "Power symbol creates a global label with name \"GND\" , ground"
-			(at 179.07 119.38 0)
-			(effects
-				(font
+			(at 176.53 119.38 0)
+			(effects
+				(font
