File: PCB/MCU.kicad_sch (KiCad schematic)
At the start: 1 part, among them U1 STM32G0B1RCTx

Commit message: Updated PCB
Changed lines of the file:
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@@
+		)
+	)
+	(hierarchical_label "MISO_BMP280"
+		(shape input)
+		(at 52.07 215.9 0)
+		(fields_autoplaced yes)
+		(effects
+			(font
+				(size 1.27 1.27)
+			)
+			(justify left)
 		)
 	)
@@
 		(shape output)
 		(at 20.32 80.01 0)
+		(fields_autoplaced yes)
+		(effects
+			(font
+				(size 1.27 1.27)
+			)
+			(justify left)
+		)
+	)
+	(hierarchical_label "CLK_BMP280"
+		(shape output)
+		(at 53.34 220.98 0)
 		(fields_autoplaced yes)
 		(effects
@@
 		)
 	)
+	(hierarchical_label "nCSS_BMP280"
+		(shape output)
+		(at 52.07 212.09 0)
+		(fields_autoplaced yes)
+		(effects
+			(font
+				(size 1.27 1.27)
+			)
+			(justify left)
+		)
+	)
 	(hierarchical_label "CLK_MPU9250"
 		(shape output)
@@
 		)
 	)
+	(hierarchical_label "MOSI_BMP280"
+		(shape output)
+		(at 52.07 218.44 0)
+		(fields_autoplaced yes)
+		(effects
+			(font
+				(size 1.27 1.27)
+			)
+			(justify left)
+		)
+	)

Commit message: Updated PCB. Added Debug section and rectifed RS485
Changed lines of the file:
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@@
 	(generator_version "8.0")
 	(paper "A4" portrait)
+	(hierarchical_label "SWO"
+		(shape bidirectional)
+		(at 109.22 236.22 0)
+		(fields_autoplaced yes)
+		(effects
+			(font
+				(size 1.27 1.27)
+			)
+			(justify left)
+		)
+	)
 	(hierarchical_label "CLK_GNSS"
 		(shape output)
@@
 		)
 	)
+	(hierarchical_label "SWCLK"
+		(shape input)
+		(at 109.22 231.14 0)
+		(fields_autoplaced yes)
+		(effects
+			(font
+				(size 1.27 1.27)
+			)
+			(justify left)
+		)
+	)
 	(hierarchical_label "CAN_SHUTDOWN"
 		(shape output)
@@
 		)
 	)
+	(hierarchical_label "SWDIO"
+		(shape bidirectional)
+		(at 109.22 233.68 0)
+		(fields_autoplaced yes)
+		(effects
+			(font
+				(size 1.27 1.27)
+			)
+			(justify left)
+		)
+	)
 	(hierarchical_label "MOSI_MPU9250"
 		(shape output)
@@
 		)
 	)
+	(hierarchical_label "RXD_RS485"
+		(shape input)
+		(at 176.53 132.08 180)
+		(fields_autoplaced yes)
+		(effects
+			(font
+				(size 1.27 1.27)
+			)
+			(justify right)
+		)
+	)
 	(hierarchical_label "3D_FIX"
 		(shape input)
@@
 		(fields_autoplaced yes)
 		(effects
+			(font
+				(size 1.27 1.27)
+			)
+			(justify left)
+		)
+	)
+	(hierarchical_label "TXD_RS485"
+		(shape output)
+		(at 176.53 154.94 180)
+		(fields_autoplaced yes)
+		(effects
+			(font
+				(size 1.27 1.27)
+			)
+			(justify right)
+		)
+	)
+	(hierarchical_label "nRESET"
+		(shape input)
+		(at 109.22 226.06 0)
+		(fields_autoplaced yes)
+		(effects

Commit message: Updated PCB.
Parts:
- renumbered U1 to U3
Changed lines of the file:
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@@
 		(dnp no)
 		(fields_autoplaced yes)
-		(property "Reference" "U1"
+		(property "Reference" "U3"
 			(at 110.1441 179.07 0)
 			(effects
@@
 		(instances
 			(project "IMU_V100"
-				(path "/b6a8d14b-6e32-4628-bf0c-2046877d1cfa/93d4a6d7-53e9-480c-99e3-973e68fe6426"
-					(reference "U1")
+				(path "/b6a8d14b-6e32-4628-bf0c-2046877d1cfa/205555cc-3b86-4915-975e-3a7e3eed6661/749fc824-56f7-4acb-b075-16c52a8f4b5a"
+					(reference "U3")
 					(unit 1)
 				)

Commit message: Updated PCB
Changed lines of the file:
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@@
+		)
+	)
+	(hierarchical_label "CAN_USER1"
+		(shape bidirectional)
+		(at 161.29 58.42 180)
+		(fields_autoplaced yes)
+		(effects
+			(font
+				(size 1.27 1.27)
+			)
+			(justify right)
 		)
 	)
@@
 		)
 	)
+	(hierarchical_label "RS485_USER2"
+		(shape bidirectional)
+		(at 176.53 137.16 180)
+		(fields_autoplaced yes)
+		(effects
+			(font
+				(size 1.27 1.27)
+			)
+			(justify right)
+		)
+	)
+	(hierarchical_label "CAN_USER2"
+		(shape bidirectional)
+		(at 161.29 60.96 180)
+		(fields_autoplaced yes)
+		(effects
+			(font
+				(size 1.27 1.27)
+			)
+			(justify right)
+		)
+	)
 	(hierarchical_label "I2C_SDA_GNSS"
 		(shape bidirectional)
@@
 	(hierarchical_label "CAN_SHUTDOWN"
 		(shape output)
-		(at 168.91 184.15 180)
+		(at 161.29 55.88 180)
 		(fields_autoplaced yes)
 		(effects
@@
 	(hierarchical_label "CAN_TX"
 		(shape output)
-		(at 168.91 179.07 180)
+		(at 161.29 50.8 180)
 		(fields_autoplaced yes)
 		(effects
@@
 	(hierarchical_label "TXD_RS485"
 		(shape output)
-		(at 176.53 154.94 180)
+		(at 176.53 134.62 180)
 		(fields_autoplaced yes)
 		(effects
@@
 		)
 	)
+	(hierarchical_label "RS485_USER1"
+		(shape bidirectional)
+		(at 176.53 129.54 180)
+		(fields_autoplaced yes)
+		(effects
+			(font
+				(size 1.27 1.27)
+			)
+			(justify right)
+		)
+	)
 	(hierarchical_label "CAN_RX"
 		(shape input)
-		(at 168.91 181.61 180)
-		(fields_autoplaced yes)
-		(effects
+		(at 161.29 53.34 180)
+		(fields_autoplaced yes)
+		(effects
