File: PCB/MCU.kicad_sch (KiCad schematic)
At the start: 1 part, among them U3 STM32G0B1RCTx

Commit message: Updated PCB
Parts:
- added C20, C21, C22, C23: C, symbol Device:C
- added Y1, Y2: Crystal_GND23, symbol Device:Crystal_GND23
Connections:
- net 3V3: now also U3.6 (VBAT), U3.7 (VREF+), U3.8 (VDD)
- net SWCLK: now also U3.46 (PA14)
- net SWDIO: now also U3.45 (PA13)
- net nRESET: now also U3.12 (PF2)
- net OSC8_IN: now reaches U3.10 (PF0)
- net OSC8_IN: now also C20.2, Y1.1
- net OSC8_OUT: now reaches U3.11 (PF1)
- net OSC8_OUT: now also C21.2, Y1.4
- net OSC32_IN: now reaches U3.4 (PC14)
- net OSC32_IN: now also C22.2, Y2.1
- net OSC32_OUT: now reaches U3.5 (PC15)
- net OSC32_OUT: now also C23.2, Y2.4
- net GND: now reaches U3.9 (VSS)
- net GND: now also C20.1, C21.1, C22.1, C23.1, Y1.2, Y1.3, Y2.2, Y2.3
Other:
- moved on the sheet: U3
