File: PCB/Project_Architecture.kicad_sch (KiCad schematic)
At the start: 0 parts

Commit message: Updated PCB.
Other:
- note added: "DEBUG"
- note added: "I2C"
- note added: "POWER"
- note added: "SIGNALS"
- note added: "SPI"
- note added: "UART"
Changed lines of the file:
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@@
+		)
+	)
+	(rectangle
+		(start 272.542 41.656)
+		(end 277.622 46.736)
+		(stroke
+			(width 0)
+			(type default)
+		)
+		(fill
+			(type color)
+			(color 194 0 194 1)
+		)
+	)
+	(rectangle
+		(start 272.542 34.036)
+		(end 277.622 39.116)
+		(stroke
+			(width 0)
+			(type default)
+		)
+		(fill
+			(type color)
+			(color 0 72 0 1)
+		)
+	)
+	(rectangle
+		(start 272.542 49.911)
+		(end 277.622 54.991)
+		(stroke
+			(width 0)
+			(type default)
+		)
+		(fill
+			(type color)
+			(color 128 77 0 1)
+		)
+	)
+	(rectangle
+		(start 272.542 26.416)
+		(end 277.622 31.496)
+		(stroke
+			(width 0)
+			(type default)
+		)
+		(fill
+			(type color)
+			(color 0 255 255 1)
+		)
+	)
+	(rectangle
+		(start 273.05 19.05)
+		(end 278.13 24.13)
+		(stroke
+			(width 0)
+			(type default)
+		)
+		(fill
+			(type color)
+			(color 194 0 0 1)
+		)
+	)
+	(rectangle
+		(start 272.542 58.166)
+		(end 277.622 63.246)
+		(stroke
+			(width 0)
+			(type default)
+		)
+		(fill
+			(type color)
+			(color 255 153 0 1)
+		)
+	)
+	(text "SPI\n"
+		(exclude_from_sim no)
+		(at 267.97 29.21 0)
+		(effects
+			(font
+				(size 1.27 1.27)
+			)
+		)
+	)
+	(text "I2C"
+		(exclude_from_sim no)
+		(at 267.97 44.45 0)
+		(effects
+			(font
+				(size 1.27 1.27)
+			)
+		)
+	)
+	(text "DEBUG\n"
+		(exclude_from_sim no)
+		(at 267.97 60.96 0)
+		(effects
+			(font
+				(size 1.27 1.27)
+			)
+		)
+	)
+	(text "UART"
+		(exclude_from_sim no)
+		(at 267.97 52.705 0)
+		(effects
+			(font
+				(size 1.27 1.27)
+			)
+		)
+	)
+	(text "POWER"
+		(exclude_from_sim no)
+		(at 268.478 21.844 0)
+		(effects
+			(font
+				(size 1.27 1.27)
+			)
+		)
+	)
+	(text "SIGNALS"
+		(exclude_from_sim no)
+		(at 267.97 36.83 0)
+		(effects
+			(font
+				(size 1.27 1.27)
+			)
 		)
 	)

Commit message: Updated PCB
Other:
- sheet CAN_FD ports: added CAN_USER1, CAN_USER2; removed none
- sheet MCU ports: added CAN_USER1, CAN_USER2, RS485_USER1, RS485_USER2; removed none
- sheet RS485_TRX ports: added RS485_USER1, RS485_USER2; removed none
Changed lines of the file:
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@@
 		(color 0 0 0 0)
 	)
-	(bus_entry
-		(at 199.39 127)
-		(size 2.54 2.54)
+	(wire
+		(pts
+			(xy 168.91 113.03) (xy 234.95 113.03)
+		)
 		(stroke
 			(width 0)
@@
 	(wire
 		(pts
-			(xy 54.61 144.78) (xy 116.84 144.78)
+			(xy 95.25 157.48) (xy 116.84 157.48)
+		)
+		(stroke
+			(width 0)
+			(type default)
+			(color 0 255 255 1)
+		)
+	)
+	(wire
+		(pts
+			(xy 102.87 137.16) (xy 54.61 137.16)
 		)
 		(stroke
@@
 	(wire
 		(pts
-			(xy 54.61 142.24) (xy 116.84 142.24)
+			(xy 97.79 154.94) (xy 116.84 154.94)
 		)
 		(stroke
@@
 	(wire
 		(pts
+			(xy 100.33 152.4) (xy 100.33 139.7)
+		)
+		(stroke
+			(width 0)
+			(type default)
+			(color 0 255 255 1)
+		)
+	)
+	(wire
+		(pts
 			(xy 24.13 161.29) (xy 30.48 161.29)
 		)
@@
 	(wire
 		(pts
+			(xy 168.91 152.4) (xy 234.95 152.4)
+		)
+		(stroke
+			(width 0)
+			(type default)
+		)
+	)
+	(wire
+		(pts
 			(xy 48.26 41.91) (xy 128.27 41.91)
 		)
@@
 	(wire
 		(pts
+			(xy 168.91 154.94) (xy 234.95 154.94)
+		)
+		(stroke
+			(width 0)
+			(type default)
+		)
+	)
+	(wire
+		(pts
 			(xy 168.91 110.49) (xy 234.95 110.49)
 		)
@@
 	(wire
 		(pts
+			(xy 168.91 115.57) (xy 234.95 115.57)
+		)
+		(stroke
+			(width 0)
+			(type default)
+		)
+	)
+	(wire
+		(pts
 			(xy 82.55 96.52) (xy 82.55 123.19)
 		)
@@
 	(wire
 		(pts
-			(xy 54.61 134.62) (xy 116.84 134.62)
+			(xy 105.41 147.32) (xy 116.84 147.32)
 		)
 		(stroke
@@
 	(wire
 		(pts
+			(xy 105.41 134.62) (xy 54.61 134.62)
+		)
+		(stroke
+			(width 0)
+			(type default)
+			(color 0 255 255 1)
+		)
+	)
+	(wire
+		(pts
+			(xy 97.79 154.94) (xy 97.79 142.24)
+		)
+		(stroke
+			(width 0)
+			(type default)
+			(color 0 255 255 1)
+		)
+	)
+	(wire
+		(pts
 			(xy 55.88 170.18) (xy 116.84 170.18)
 		)
@@
 	(wire
 		(pts
-			(xy 54.61 137.16) (xy 116.84 137.16)
+			(xy 95.25 157.48) (xy 95.25 144.78)
+		)
+		(stroke
+			(width 0)
+			(type default)
+			(color 0 255 255 1)
+		)
+	)
+	(wire
+		(pts
+			(xy 102.87 149.86) (xy 116.84 149.86)
 		)
 		(stroke
@@
 	(wire
 		(pts
+			(xy 97.79 142.24) (xy 54.61 142.24)
+		)
+		(stroke
+			(width 0)
+			(type default)
+			(color 0 255 255 1)
+		)
+	)
+	(wire
+		(pts
 			(xy 55.88 101.6) (xy 77.47 101.6)
 		)
@@
 	(wire
 		(pts
-			(xy 54.61 139.7) (xy 116.84 139.7)
+			(xy 100.33 152.4) (xy 116.84 152.4)
 		)
 		(stroke
@@
 	(wire
 		(pts
+			(xy 105.41 147.32) (xy 105.41 134.62)
+		)
+		(stroke
+			(width 0)
+			(type default)
+			(color 0 255 255 1)
+		)
+	)
+	(wire
+		(pts
+			(xy 95.25 144.78) (xy 54.61 144.78)
+		)
+		(stroke
+			(width 0)
+			(type default)
+			(color 0 255 255 1)
+		)
+	)
+	(wire
+		(pts
+			(xy 100.33 139.7) (xy 54.61 139.7)
+		)
+		(stroke
+			(width 0)
+			(type default)
+			(color 0 255 255 1)
+		)
+	)
+	(wire
+		(pts
 			(xy 95.25 110.49) (xy 116.84 110.49)
 		)
@@
 			(type default)
 			(color 128 77 0 1)
+		)
+	)
+	(wire
+		(pts
+			(xy 102.87 149.86) (xy 102.87 137.16)
+		)
+		(stroke
+			(width 0)
+			(type default)
+			(color 0 255 255 1)
 		)
 	)
@@
 			)
 		)
+		(pin "CAN_USER2" bidirectional
+			(at 234.95 154.94 180)
+			(effects
+				(font
+					(size 1.27 1.27)
+				)
+				(justify left)
+			)
+		)
+		(pin "CAN_USER1" bidirectional
+			(at 234.95 152.4 180)
+			(effects
+				(font
+					(size 1.27 1.27)
+				)
+				(justify left)
+			)
+		)
 		(instances
 			(project "IMU_V100"
@@
 		)
 		(pin "MISO_MPU9250" input
-			(at 116.84 139.7 180)
+			(at 116.84 152.4 180)
 			(effects
 				(font
@@
 		)
 		(pin "MOSI_MPU9250" output
-			(at 116.84 137.16 180)
+			(at 116.84 149.86 180)
 			(effects
 				(font
@@
 		)
 		(pin "INT_MPU9250" input
-			(at 116.84 144.78 180)
+			(at 116.84 157.48 180)
 			(effects
 				(font
@@
 		)
 		(pin "nCSS_MPU9250" output
-			(at 116.84 134.62 180)
+			(at 116.84 147.32 180)
 			(effects
 				(font
@@
 		)
 		(pin "CLK_MPU9250" output
-			(at 116.84 142.24 180)
+			(at 116.84 154.94 180)
 			(effects
 				(font
@@
 		(pin "SWCLK" input
 			(at 130.81 82.55 90)
+			(effects
+				(font
+					(size 1.27 1.27)
+				)
+				(justify right)
+			)
+		)
+		(pin "CAN_USER1" bidirectional
+			(at 168.91 152.4 0)
+			(effects
+				(font
+					(size 1.27 1.27)
+				)
+				(justify right)
+			)
+		)
+		(pin "CAN_USER2" bidirectional
+			(at 168.91 154.94 0)
+			(effects
+				(font
+					(size 1.27 1.27)
+				)
+				(justify right)
+			)
+		)
+		(pin "RS485_USER1" bidirectional
+			(at 168.91 113.03 0)
+			(effects
+				(font
+					(size 1.27 1.27)
+				)
+				(justify right)
+			)
+		)
+		(pin "RS485_USER2" bidirectional
+			(at 168.91 115.57 0)
 			(effects
 				(font
@@
 			(effects
 				(font
+					(size 1.27 1.27)
+				)
+				(justify left)
+			)
+		)
+		(pin "RS485_USER2" bidirectional
+			(at 234.95 113.03 180)
+			(effects
+				(font
+					(size 1.27 1.27)
+				)
+				(justify left)
+			)
+		)
+		(pin "RS485_USER1" bidirectional
+			(at 234.95 115.57 180)
+			(effects
+				(font
