File: PCB/Project_Architecture.kicad_sch (KiCad schematic)
At the start: 0 parts

Commit message: Updated PCB
Parts:
- added H2, H3, H4, Hd1: MountingHole, MountingHole:MountingHole_3.2mm_M3_DIN965, symbol Mechanical:MountingHole

Commit message: Updated PCB
Parts:
- renumbered H2 to H1, H3 to H2, H4 to H3
Changed lines of the file:
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@@
 		(dnp no)
 		(fields_autoplaced yes)
-		(property "Reference" "H3"
+		(property "Reference" "H2"
 			(at 228.6 171.4499 0)
 			(effects
@@
 			(project "IMU_V100"
 				(path "/b6a8d14b-6e32-4628-bf0c-2046877d1cfa/205555cc-3b86-4915-975e-3a7e3eed6661"
-					(reference "H3")
+					(reference "H2")
 					(unit 1)
 				)
@@
 		(dnp no)
 		(fields_autoplaced yes)
-		(property "Reference" "H2"
+		(property "Reference" "H1"
 			(at 209.55 171.4499 0)
 			(effects
@@
 			(project "IMU_V100"
 				(path "/b6a8d14b-6e32-4628-bf0c-2046877d1cfa/205555cc-3b86-4915-975e-3a7e3eed6661"
-					(reference "H2")
+					(reference "H1")
 					(unit 1)
 				)
@@
 		(dnp no)
 		(fields_autoplaced yes)
-		(property "Reference" "H4"
+		(property "Reference" "H3"
 			(at 247.65 171.4499 0)
 			(effects
@@
 			(project "IMU_V100"
 				(path "/b6a8d14b-6e32-4628-bf0c-2046877d1cfa/205555cc-3b86-4915-975e-3a7e3eed6661"
-					(reference "H4")
+					(reference "H3")
 					(unit 1)
 				)
