File: PCB/IMU_V100.kicad_pcb (KiCad board)
At the start: 2 copper layers, 89 x 44 mm, 16 parts, among them IC1 LC76GABMD, J1 1-770969-0, J2 Conn_ARM_SWD_TagConnect_TC2030, J4 1-770969-0, U1 BMP280, U2 MCP2557FD-xMNY, U3 STM32G0B1RCTx, U4 XL1509-3.3, U5 SN65HVD11HD

Commit message: Updated PCB
Parts:
- removed D5, D6: PTVS3V3S1UTR, PCM_Diode_SMD_AKL:D_SOD-123F
- removed D7: SM712, PCM_Package_TO_SOT_SMD_AKL:SOT-23
- removed U4: XL1509-3.3, Package_SO:SOIC-8_3.9x4.9mm_P1.27mm
- added C10: C, Capacitor_SMD:C_0402_1005Metric_Pad0.74x0.62mm_HandSolder, B.Cu at (146.0, 64.1)
- added C11: 100nF, Capacitor_SMD:C_0402_1005Metric_Pad0.74x0.62mm_HandSolder, B.Cu at (146.0, 62.1)
- added C12: 33pF, Capacitor_SMD:C_0402_1005Metric_Pad0.74x0.62mm_HandSolder, B.Cu at (146.0, 60.1)
- added C13: C, Capacitor_SMD:C_0402_1005Metric_Pad0.74x0.62mm_HandSolder, B.Cu at (146.0, 58.2)
- added C19: 0.1uF, Capacitor_SMD:C_0603_1608Metric_Pad1.08x0.95mm_HandSolder, F.Cu at (171.2, 119.8)
- added C20: 4700pF, Capacitor_SMD:C_0603_1608Metric_Pad1.08x0.95mm_HandSolder, F.Cu at (171.0, 128.6)
- added C5: 10uF, Capacitor_SMD:C_0402_1005Metric_Pad0.74x0.62mm_HandSolder, B.Cu at (146.0, 73.9)
- added C6: 100nF, Capacitor_SMD:C_0402_1005Metric_Pad0.74x0.62mm_HandSolder, B.Cu at (146.0, 72.0)
- added C7: C, Capacitor_SMD:C_0402_1005Metric_Pad0.74x0.62mm_HandSolder, B.Cu at (146.0, 70.0)
- added C8: 10uF, Capacitor_SMD:C_0402_1005Metric_Pad0.74x0.62mm_HandSolder, B.Cu at (146.0, 68.0)
- added C9: 33pF, Capacitor_SMD:C_0402_1005Metric_Pad0.74x0.62mm_HandSolder, B.Cu at (146.0, 66.0)
- added H2: MountingHole, MountingHole:MountingHole_3.2mm_M3_DIN965, F.Cu at (185.0, 92.0)
- added H3: MountingHole, MountingHole:MountingHole_3.2mm_M3_DIN965, F.Cu at (132.0, 140.0)
- added H4: MountingHole, MountingHole:MountingHole_3.2mm_M3_DIN965, F.Cu at (185.0, 140.0)
- added Hd1: MountingHole, MountingHole:MountingHole_3.2mm_M3_DIN965, F.Cu at (132.0, 92.0)
- added R10: 2.2K, Resistor_SMD:R_0402_1005Metric, B.Cu at (128.0, 79.0)
- added R11: 10K, Resistor_SMD:R_0402_1005Metric, B.Cu at (116.4, 70.1)
- added R18: 60R, Resistor_SMD:R_0603_1608Metric_Pad0.98x0.95mm_HandSolder, F.Cu at (173.0, 126.8)
- added R19: 60R, Resistor_SMD:R_0603_1608Metric_Pad0.98x0.95mm_HandSolder, F.Cu at (169.4, 126.8)
- added R4: R, Resistor_SMD:R_0402_1005Metric, B.Cu at (155.9, 78.0)
- added R5: R, Resistor_SMD:R_0402_1005Metric, B.Cu at (155.9, 76.0)
- added R6: 0R, Resistor_SMD:R_0402_1005Metric, B.Cu at (110.7, 72.8)
- added R7: 0R, Resistor_SMD:R_0402_1005Metric, B.Cu at (126.4, 79.4)
- added R8: 0R, Resistor_SMD:R_0402_1005Metric, B.Cu at (126.4, 80.6)
- added R9: 2.2K, Resistor_SMD:R_0402_1005Metric, B.Cu at (128.0, 81.2)
- added U6: THVD1450DR, Package_SON:VSON-8-1EP_3x3mm_P0.65mm_EP1.6x2.4mm, F.Cu at (146.0, 125.6)
- IC1: moved to B.Cu
- U5: value SN65HVD11HD -> TPS62933; footprint Package_SO:SOIC-8_3.9x4.9mm_P1.27mm -> Package_TO_SOT_SMD:SOT-583-8
- moved U2 130.2 mm to (171.2, 122.8), turned to -90 degrees
- moved U1 121.3 mm to (175.2, 106.0)
- moved U5 111.4 mm to (116.7, 138.3)
- moved IC1 83.3 mm to (140.2, 108.8), turned to 180 degrees
- moved D1 65.1 mm to (109.0, 125.8)
- moved D2 65.1 mm to (109.0, 128.2)
- moved D3 65.1 mm to (109.0, 130.7)
- moved D4 65.1 mm to (109.0, 133.1)
- moved J4 55.7 mm to (150.1, 131.5), turned to 0 degrees
- moved J2 34.9 mm to (177.5, 91.0)
- moved J1 23.7 mm to (175.1, 131.5), turned to 0 degrees
- moved U3 20.0 mm to (160.0, 100.0)
Connections:
- J1 pad 3: unconnected-(J1-Pad3) -> /Project_Architecture/CAN_FD/CAN_USER1
- J1 pad 6: unconnected-(J1-Pad6) -> /Project_Architecture/CAN_FD/CAN_USER2
- J4 pad 3: unconnected-(J4-Pad3) -> /Project_Architecture/MCU/RS485_USER2
- J4 pad 6: unconnected-(J4-Pad6) -> /Project_Architecture/MCU/RS485_USER1
- U5 pad 1: /Project_Architecture/MCU/RXD_RS485 -> unconnected-(U5-RT-Pad1)
- U5 pad 2: Net-(R15-+) -> Net-(U5-EN)
- U5 pad 3: Net-(R15-+) -> /Project_Architecture/CAN_FD/VIN
- U5 pad 4: /Project_Architecture/MCU/TXD_RS485 -> GND
- U5 pad 5: unconnected-(U5-GND-Pad5) -> Net-(U5-SW)
- U5 pad 8: +3V3 -> Net-(U5-FB)
Routing:
- net Net-(R19-+): track 0.00 -> 14.4 mm
- net Net-(R18--): track 0.00 -> 10.3 mm
- net GND: track 0.00 -> 4.76 mm, vias 0 -> 2
- net Net-(C20--): track 0.00 -> 3.67 mm
- net +3V3: track 0.00 -> 1.80 mm
Other:
- board size 89 x 44 mm -> 64 x 59 mm

Commit message: Updated  Pcb
Parts:
- moved U5 46.9 mm to (160.9, 122.5)
- moved D1 46.9 mm to (153.1, 110.0)
- moved D2 46.9 mm to (153.1, 112.4)
- moved D3 46.9 mm to (153.1, 114.9)
- moved D4 46.9 mm to (153.1, 117.3)
- moved R11 36.5 mm to (141.8, 96.3)
- moved R6 36.5 mm to (136.1, 99.0)
- moved C10 31.4 mm to (150.4, 95.2)
- moved C11 31.4 mm to (150.4, 93.2)
- moved C6 31.4 mm to (150.4, 103.0)
- moved C7 31.4 mm to (150.4, 101.1)
- moved C8 31.4 mm to (150.4, 99.1)
- moved C9 31.4 mm to (150.4, 97.1)
- moved C12 31.4 mm to (150.4, 91.2)
- moved C13 31.4 mm to (150.4, 89.2)
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Changed lines of the file:
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@@
 	(footprint "Diode_SMD:D_SOD-523"
 		(layer "F.Cu")
-		(at 108.95 128.21)
+		(at 153.105 112.425)
 		(descr "http://www.diodes.com/datasheets/ap02001.pdf p.144")
 		(tags "Diode SOD523")
@@
 	(footprint "Diode_SMD:D_SOD-523"
 		(layer "F.Cu")
-		(at 108.95 125.76)
+		(at 153.105 109.975)
 		(descr "http://www.diodes.com/datasheets/ap02001.pdf p.144")
 		(tags "Diode SOD523")
@@
 	(footprint "Diode_SMD:D_SOD-523"
 		(layer "F.Cu")
-		(at 108.95 133.11)
+		(at 153.105 117.325)
 		(descr "http://www.diodes.com/datasheets/ap02001.pdf p.144")
 		(tags "Diode SOD523")
@@
 	(footprint "Package_TO_SOT_SMD:SOT-583-8"
 		(layer "F.Cu")
-		(at 116.705 138.335)
+		(at 160.86 122.55)
 		(descr "https://www.ti.com/lit/ds/symlink/tps62933.pdf")
 		(tags "SOT-583-8")
@@
 	(footprint "Diode_SMD:D_SOD-523"
 		(layer "F.Cu")
-		(at 108.95 130.66)
+		(at 153.105 114.875)
 		(descr "http://www.diodes.com/datasheets/ap02001.pdf p.144")
 		(tags "Diode SOD523")
@@
 	(footprint "Capacitor_SMD:C_0402_1005Metric_Pad0.74x0.62mm_HandSolder"
 		(layer "B.Cu")
-		(at 146.0325 64.08)
+		(at 150.4 95.15)
 		(descr "Capacitor SMD 0402 (1005 Metric), square (rectangular) end terminal, IPC_7351 nominal with elongated pad for handsoldering. (Body size source: IPC-SM-782 page 76, https://www.pcb-3d.com/wordpress/wp-content/uploads/ipc-sm-782a_amendment_1_and_2.pdf), generated with kicad-footprint-generator")
 		(tags "capacitor handsolder")
@@
 	(footprint "Resistor_SMD:R_0402_1005Metric"
 		(layer "B.Cu")
-		(at 155.89 78)
+		(at 145.29 92.6)
 		(descr "Resistor SMD 0402 (1005 Metric), square (rectangular) end terminal, IPC_7351 nominal, (Body size source: IPC-SM-782 page 72, https://www.pcb-3d.com/wordpress/wp-content/uploads/ipc-sm-782a_amendment_1_and_2.pdf), generated with kicad-footprint-generator")
 		(tags "resistor")
@@
 	(footprint "Resistor_SMD:R_0402_1005Metric"
 		(layer "B.Cu")
-		(at 128 81.17 90)
+		(at 140 91.8 90)
 		(descr "Resistor SMD 0402 (1005 Metric), square (rectangular) end terminal, IPC_7351 nominal, (Body size source: IPC-SM-782 page 72, https://www.pcb-3d.com/wordpress/wp-content/uploads/ipc-sm-782a_amendment_1_and_2.pdf), generated with kicad-footprint-generator")
 		(tags "resistor")
@@
 		)
 		(property "Datasheet" ""
-			(at 0 0 -90)
+			(at 0 0 270)
 			(unlocked yes)
 			(layer "B.Fab")
@@
 		)
 		(property "Description" "resistor"
-			(at 0 0 -90)
+			(at 0 0 270)
 			(unlocked yes)
 			(layer "B.Fab")
@@
 		)
 		(property "Indicator" "+"
-			(at 0 0 -90)
+			(at 0 0 270)
 			(unlocked yes)
 			(layer "B.Fab")
@@
 		)
 		(property "Rating" "W"
-			(at 0 0 -90)
+			(at 0 0 270)
 			(unlocked yes)
 			(layer "B.Fab")
@@
 	(footprint "Capacitor_SMD:C_0402_1005Metric_Pad0.74x0.62mm_HandSolder"
 		(layer "B.Cu")
-		(at 146.0325 66.05)
+		(at 150.4 97.12)
 		(descr "Capacitor SMD 0402 (1005 Metric), square (rectangular) end terminal, IPC_7351 nominal with elongated pad for handsoldering. (Body size source: IPC-SM-782 page 76, https://www.pcb-3d.com/wordpress/wp-content/uploads/ipc-sm-782a_amendment_1_and_2.pdf), generated with kicad-footprint-generator")
 		(tags "capacitor handsolder")
@@
 	(footprint "Resistor_SMD:R_0402_1005Metric"
 		(layer "B.Cu")
-		(at 116.4 70.06 -90)
+		(at 141.8 96.29 -90)
 		(descr "Resistor SMD 0402 (1005 Metric), square (rectangular) end terminal, IPC_7351 nominal, (Body size source: IPC-SM-782 page 72, https://www.pcb-3d.com/wordpress/wp-content/uploads/ipc-sm-782a_amendment_1_and_2.pdf), generated with kicad-footprint-generator")
 		(tags "resistor")
@@
 	(footprint "Capacitor_SMD:C_0402_1005Metric_Pad0.74x0.62mm_HandSolder"
 		(layer "B.Cu")
-		(at 146.0325 68.02)
+		(at 150.4 99.09)
 		(descr "Capacitor SMD 0402 (1005 Metric), square (rectangular) end terminal, IPC_7351 nominal with elongated pad for handsoldering. (Body size source: IPC-SM-782 page 76, https://www.pcb-3d.com/wordpress/wp-content/uploads/ipc-sm-782a_amendment_1_and_2.pdf), generated with kicad-footprint-generator")
 		(tags "capacitor handsolder")
@@
 	(footprint "Capacitor_SMD:C_0402_1005Metric_Pad0.74x0.62mm_HandSolder"
 		(layer "B.Cu")
-		(at 146.0325 60.14)
+		(at 150.4 91.21)
 		(descr "Capacitor SMD 0402 (1005 Metric), square (rectangular) end terminal, IPC_7351 nominal with elongated pad for handsoldering. (Body size source: IPC-SM-782 page 76, https://www.pcb-3d.com/wordpress/wp-content/uploads/ipc-sm-782a_amendment_1_and_2.pdf), generated with kicad-footprint-generator")
 		(tags "capacitor handsolder")
@@
 	(footprint "Resistor_SMD:R_0402_1005Metric"
 		(layer "B.Cu")
-		(at 126.4 79.37)
+		(at 138.4 90)
 		(descr "Resistor SMD 0402 (1005 Metric), square (rectangular) end terminal, IPC_7351 nominal, (Body size source: IPC-SM-782 page 72, https://www.pcb-3d.com/wordpress/wp-content/uploads/ipc-sm-782a_amendment_1_and_2.pdf), generated with kicad-footprint-generator")
 		(tags "resistor")
@@
 	(footprint "Capacitor_SMD:C_0402_1005Metric_Pad0.74x0.62mm_HandSolder"
 		(layer "B.Cu")
-		(at 146.0325 58.17)
+		(at 150.4 89.24)
 		(descr "Capacitor SMD 0402 (1005 Metric), square (rectangular) end terminal, IPC_7351 nominal with elongated pad for handsoldering. (Body size source: IPC-SM-782 page 76, https://www.pcb-3d.com/wordpress/wp-content/uploads/ipc-sm-782a_amendment_1_and_2.pdf), generated with kicad-footprint-generator")
 		(tags "capacitor handsolder")
@@
 	(footprint "Resistor_SMD:R_0402_1005Metric"
 		(layer "B.Cu")
-		(at 126.4 80.57)
+		(at 138.4 91.2)
 		(descr "Resistor SMD 0402 (1005 Metric), square (rectangular) end terminal, IPC_7351 nominal, (Body size source: IPC-SM-782 page 72, https://www.pcb-3d.com/wordpress/wp-content/uploads/ipc-sm-782a_amendment_1_and_2.pdf), generated with kicad-footprint-generator")
 		(tags "resistor")
@@
 	(footprint "Resistor_SMD:R_0402_1005Metric"
 		(layer "B.Cu")
-		(at 155.89 76.01)
+		(at 145.29 90.61)
 		(descr "Resistor SMD 0402 (1005 Metric), square (rectangular) end terminal, IPC_7351 nominal, (Body size source: IPC-SM-782 page 72, https://www.pcb-3d.com/wordpress/wp-content/uploads/ipc-sm-782a_amendment_1_and_2.pdf), generated with kicad-footprint-generator")
 		(tags "resistor")
@@
 	(footprint "Capacitor_SMD:C_0402_1005Metric_Pad0.74x0.62mm_HandSolder"
 		(layer "B.Cu")
-		(at 146.0325 71.96)
+		(at 150.4 103.03)
 		(descr "Capacitor SMD 0402 (1005 Metric), square (rectangular) end terminal, IPC_7351 nominal with elongated pad for handsoldering. (Body size source: IPC-SM-782 page 76, https://www.pcb-3d.com/wordpress/wp-content/uploads/ipc-sm-782a_amendment_1_and_2.pdf), generated with kicad-footprint-generator")
 		(tags "capacitor handsolder")
@@
 	(footprint "Capacitor_SMD:C_0402_1005Metric_Pad0.74x0.62mm_HandSolder"
 		(layer "B.Cu")
-		(at 146.0325 62.11)
+		(at 150.4 93.18)
 		(descr "Capacitor SMD 0402 (1005 Metric), square (rectangular) end terminal, IPC_7351 nominal with elongated pad for handsoldering. (Body size source: IPC-SM-782 page 76, https://www.pcb-3d.com/wordpress/wp-content/uploads/ipc-sm-782a_amendment_1_and_2.pdf), generated with kicad-footprint-generator")
 		(tags "capacitor handsolder")
@@
 	(footprint "Capacitor_SMD:C_0402_1005Metric_Pad0.74x0.62mm_HandSolder"
 		(layer "B.Cu")
-		(at 146.0325 69.99)
+		(at 150.4 101.06)
 		(descr "Capacitor SMD 0402 (1005 Metric), square (rectangular) end terminal, IPC_7351 nominal with elongated pad for handsoldering. (Body size source: IPC-SM-782 page 76, https://www.pcb-3d.com/wordpress/wp-content/uploads/ipc-sm-782a_amendment_1_and_2.pdf), generated with kicad-footprint-generator")
 		(tags "capacitor handsolder")
@@
 	(footprint "Capacitor_SMD:C_0402_1005Metric_Pad0.74x0.62mm_HandSolder"
 		(layer "B.Cu")
-		(at 146.0325 73.93)
+		(at 150.4 105)
 		(descr "Capacitor SMD 0402 (1005 Metric), square (rectangular) end terminal, IPC_7351 nominal with elongated pad for handsoldering. (Body size source: IPC-SM-782 page 76, https://www.pcb-3d.com/wordpress/wp-content/uploads/ipc-sm-782a_amendment_1_and_2.pdf), generated with kicad-footprint-generator")
 		(tags "capacitor handsolder")
@@
 	(footprint "Resistor_SMD:R_0402_1005Metric"
 		(layer "B.Cu")
-		(at 128 78.97 -90)
+		(at 140 89.6 -90)
 		(descr "Resistor SMD 0402 (1005 Metric), square (rectangular) end terminal, IPC_7351 nominal, (Body size source: IPC-SM-782 page 72, https://www.pcb-3d.com/wordpress/wp-content/uploads/ipc-sm-782a_amendment_1_and_2.pdf), generated with kicad-footprint-generator")
 		(tags "resistor")
@@
 	(footprint "Resistor_SMD:R_0402_1005Metric"
 		(layer "B.Cu")
-		(at 110.69 72.77)
+		(at 136.09 99)
 		(descr "Resistor SMD 0402 (1005 Metric), square (rectangular) end terminal, IPC_7351 nominal, (Body size source: IPC-SM-782 page 72, https://www.pcb-3d.com/wordpress/wp-content/uploads/ipc-sm-782a_amendment_1_and_2.pdf), generated with kicad-footprint-generator")
 		(tags "resistor")

Commit message: Updated PCB
Parts:
- removed C20: 4700pF, Capacitor_SMD:C_0603_1608Metric_Pad1.08x0.95mm_HandSolder
- removed H4: MountingHole, MountingHole:MountingHole_3.2mm_M3_DIN965
- removed R18, R19: 60R, Resistor_SMD:R_0603_1608Metric_Pad0.98x0.95mm_HandSolder
- removed U6: THVD1450DR, Package_SON:VSON-8-1EP_3x3mm_P0.65mm_EP1.6x2.4mm
- added C1: 4.7uF, Capacitor_SMD:C_0603_1608Metric, F.Cu at (160.3, 128.3)
- added C14: 33pF, Capacitor_SMD:C_0402_1005Metric_Pad0.74x0.62mm_HandSolder, F.Cu at (237.9, 112.5)
- added C15: C, Capacitor_SMD:C_0402_1005Metric_Pad0.74x0.62mm_HandSolder, F.Cu at (237.9, 114.5)
- added C16: 4.7uF, Capacitor_SMD:C_0603_1608Metric, F.Cu at (131.7, 120.4)
- added C17: 560nF, Capacitor_SMD:C_0603_1608Metric, F.Cu at (131.7, 122.9)
- added C18: 4.7uF, Capacitor_SMD:C_0603_1608Metric, F.Cu at (131.7, 125.4)
- added C2: 560nF, Capacitor_SMD:C_0603_1608Metric, F.Cu at (157.9, 131.0)
- added C3: 0.1uF, Capacitor_SMD:C_0603_1608Metric_Pad1.08x0.95mm_HandSolder, F.Cu at (222.8, 103.7)
- added C3: 0.1uF, Capacitor_SMD:C_0603_1608Metric_Pad1.08x0.95mm_HandSolder, F.Cu at (160.3, 125.3)
- added C4: 4700pF, Capacitor_SMD:C_0603_1608Metric_Pad1.08x0.95mm_HandSolder, F.Cu at (222.8, 106.2)
- added H1: MountingHole, MountingHole:MountingHole_3.2mm_M3_DIN965, F.Cu at (230.5, 106.0)
- added L1: 1uH, Inductor_SMD:L_0805_2012Metric_Pad1.05x1.20mm_HandSolder, F.Cu at (157.2, 125.7)
- added L2: 1uH, Inductor_SMD:L_0805_2012Metric_Pad1.05x1.20mm_HandSolder, F.Cu at (136.1, 120.5)
- added R1: 60R, Resistor_SMD:R_0603_1608Metric_Pad0.98x0.95mm_HandSolder, F.Cu at (222.8, 108.7)
- added R12: 2.2K, Resistor_SMD:R_0402_1005Metric, F.Cu at (234.9, 112.5)
- added R13: 10K, Resistor_SMD:R_0402_1005Metric, F.Cu at (234.9, 114.5)
- added R2: 60R, Resistor_SMD:R_0603_1608Metric_Pad0.98x0.95mm_HandSolder, F.Cu at (222.8, 111.2)
- added U1: BMP280, Package_LGA:Bosch_LGA-8_2x2.5mm_P0.65mm_ClockwisePinNumbering, F.Cu at (157.9, 128.9)
- added U4: MIC23050-SYML, Package_DFN_QFN:Micrel_MLF-8-1EP_2x2mm_P0.5mm_EP0.6x1.2mm_ThermalVias, F.Cu at (136.0, 123.8)
- C10, C7: value C -> 10uF
- C11: value 100nF -> 33pF
- C12, C9: value 33pF -> C
- C13: value C -> 100nF
- C8: value 10uF -> 100nF
- R10, R9: value 2.2K -> 0R
- R11: value 10K -> 2.2K
- R6, R7: value 0R -> R
- U5: value TPS62933 -> THVD1450DR; footprint Package_TO_SOT_SMD:SOT-583-8 -> Package_SON:VSON-8-1EP_3x3mm_P0.65mm_EP1.6x2.4mm
- moved U5 16.8 mm to (144.4, 125.8)
- moved U3 2.66 mm to (162.7, 100.2)
Connections:
- C10 pad 1: GND -> Net-(BT1-+)
- C10 pad 2: Net-(C10--) -> GND
- C11 pad 1: Net-(BT1-+) -> +3V3
- C12 pad 1: Net-(BT1-+) -> GND
- C12 pad 2: GND -> Net-(C12--)
- C13 pad 1: GND -> Net-(BT1-+)
- C13 pad 2: Net-(C13--) -> GND
- C7 pad 1: Net-(C7-+) -> +3V3
- C7 pad 2: Net-(C10--) -> GND
- C8 pad 1: Net-(BT1-+) -> +3V3
- C9 pad 1: +3V3 -> Net-(C9-+)
- C9 pad 2: GND -> Net-(C12--)
- IC1 pad 11: Net-(C13--) -> Net-(C15--)
- R10 pad 1: +3V3 -> Net-(IC1-I2C_SCL)
- R10 pad 2: /Project_Architecture/GPS/I2C_SDA_GNSS -> /Project_Architecture/GPS/I2C_SCL_GNSS
- R11 pad 2: Net-(IC1-RESERVED_5) -> /Project_Architecture/GPS/I2C_SCL_GNSS
- R6 pad 1: /Project_Architecture/GPS/nRESET_GNSS -> Net-(C12--)
- R6 pad 2: Net-(IC1-RESET_N) -> Net-(C15--)
- R7 pad 1: Net-(IC1-I2C_SDA) -> Net-(L1--)
- R7 pad 2: /Project_Architecture/GPS/I2C_SDA_GNSS -> Net-(IC1-VDD_RF)
- R8 pad 1: Net-(IC1-I2C_SCL) -> /Project_Architecture/GPS/nRESET_GNSS
- R8 pad 2: /Project_Architecture/GPS/I2C_SCL_GNSS -> Net-(IC1-RESET_N)
- R9 pad 1: +3V3 -> Net-(IC1-I2C_SDA)
- R9 pad 2: /Project_Architecture/GPS/I2C_SCL_GNSS -> /Project_Architecture/GPS/I2C_SDA_GNSS
- U5 pad 1: unconnected-(U5-RT-Pad1) -> /Project_Architecture/MCU/RXD_RS485
- U5 pad 2: Net-(U5-EN) -> Net-(R15-+)
- U5 pad 3: /Project_Architecture/CAN_FD/VIN -> Net-(R15-+)
- U5 pad 4: GND -> /Project_Architecture/MCU/TXD_RS485
- U5 pad 5: Net-(U5-SW) -> unconnected-(U5-GND-Pad5)
- U5 pad 8: Net-(U5-FB) -> +3V3
Routing:
- net /3V3: track 0.00 -> 8.79 mm, vias 0 -> 2
- net /VIN: track 0.00 -> 7.03 mm, vias 0 -> 2
- net Net-(C20--): track 3.67 -> 0.00 mm
- net (no net): track 0.00 -> 3.67 mm
- added copper zone on F.Cu, net /Project_Architecture/Barometer/CLK_BMP280
- added copper zone on F.Cu, net /Project_Architecture/Barometer/MOSI_BMP280
- added copper zone on F.Cu, net /Project_Architecture/Barometer/nCSS_BMP280
- added copper zone on B.Cu, net GND
- added copper zone on F.Cu, net GND
