File: PCB/RS485_TRX.kicad_sch (KiCad schematic)
At the start: 10 parts, among them J4 1-770969-0, U6 THVD1450DR

Commit message: Updated PCB
Parts:
- renumbered C18 to C19, D8 to D7, R20 to R16, R21 to R17, U6 to U5
Changed lines of the file:
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@@
 		(dnp no)
 		(fields_autoplaced yes)
-		(property "Reference" "R21"
+		(property "Reference" "R17"
 			(at 153.67 102.87 90)
 			(effects
@@
 			(project "IMU_V100"
 				(path "/b6a8d14b-6e32-4628-bf0c-2046877d1cfa/205555cc-3b86-4915-975e-3a7e3eed6661/84e3f5e1-ab68-44f3-8700-c3af58140fdb"
-					(reference "R21")
+					(reference "R17")
 					(unit 1)
 				)
@@
 		(dnp no)
 		(fields_autoplaced yes)
-		(property "Reference" "#PWR028"
+		(property "Reference" "#PWR029"
 			(at 104.14 78.74 0)
 			(effects
@@
 			(project "IMU_V100"
 				(path "/b6a8d14b-6e32-4628-bf0c-2046877d1cfa/205555cc-3b86-4915-975e-3a7e3eed6661/84e3f5e1-ab68-44f3-8700-c3af58140fdb"
-					(reference "#PWR028")
+					(reference "#PWR029")
 					(unit 1)
 				)
@@
 		(dnp no)
 		(fields_autoplaced yes)
-		(property "Reference" "#PWR029"
+		(property "Reference" "#PWR030"
 			(at 118.11 53.34 0)
 			(effects
@@
 			(project "IMU_V100"
 				(path "/b6a8d14b-6e32-4628-bf0c-2046877d1cfa/205555cc-3b86-4915-975e-3a7e3eed6661/84e3f5e1-ab68-44f3-8700-c3af58140fdb"
-					(reference "#PWR029")
+					(reference "#PWR030")
 					(unit 1)
 				)
@@
 		(dnp no)
 		(fields_autoplaced yes)
-		(property "Reference" "D8"
+		(property "Reference" "D7"
 			(at 188.6585 80.01 0)
 			(effects
@@
 			(project ""
 				(path "/b6a8d14b-6e32-4628-bf0c-2046877d1cfa/205555cc-3b86-4915-975e-3a7e3eed6661/84e3f5e1-ab68-44f3-8700-c3af58140fdb"
-					(reference "D8")
+					(reference "D7")
 					(unit 1)
 				)
@@
 		(dnp no)
 		(fields_autoplaced yes)
-		(property "Reference" "#PWR035"
+		(property "Reference" "#PWR031"
 			(at 176.53 104.14 0)
 			(effects
@@
 			(project "IMU_V100"
 				(path "/b6a8d14b-6e32-4628-bf0c-2046877d1cfa/205555cc-3b86-4915-975e-3a7e3eed6661/84e3f5e1-ab68-44f3-8700-c3af58140fdb"
-					(reference "#PWR035")
+					(reference "#PWR031")
 					(unit 1)
 				)
@@
 		(dnp no)
 		(fields_autoplaced yes)
-		(property "Reference" "U6"
+		(property "Reference" "U5"
 			(at 120.3041 80.01 0)
 			(effects
@@
 			(project ""
 				(path "/b6a8d14b-6e32-4628-bf0c-2046877d1cfa/205555cc-3b86-4915-975e-3a7e3eed6661/84e3f5e1-ab68-44f3-8700-c3af58140fdb"
-					(reference "U6")
+					(reference "U5")
 					(unit 1)
 				)
@@
 		(dnp no)
 		(fields_autoplaced yes)
-		(property "Reference" "C18"
+		(property "Reference" "C19"
 			(at 107.95 63.4999 0)
 			(effects
@@
 			(project "IMU_V100"
 				(path "/b6a8d14b-6e32-4628-bf0c-2046877d1cfa/205555cc-3b86-4915-975e-3a7e3eed6661/84e3f5e1-ab68-44f3-8700-c3af58140fdb"
-					(reference "C18")
+					(reference "C19")
 					(unit 1)
 				)
@@
 		(dnp no)
 		(fields_autoplaced yes)
-		(property "Reference" "#PWR026"
+		(property "Reference" "#PWR028"
 			(at 96.52 139.7 0)
 			(effects
@@
 			(project "IMU_V100"
 				(path "/b6a8d14b-6e32-4628-bf0c-2046877d1cfa/205555cc-3b86-4915-975e-3a7e3eed6661/84e3f5e1-ab68-44f3-8700-c3af58140fdb"
-					(reference "#PWR026")
+					(reference "#PWR028")
 					(unit 1)
 				)
@@
 		(dnp no)
 		(fields_autoplaced yes)
-		(property "Reference" "R20"
+		(property "Reference" "R16"
 			(at 153.67 71.12 90)
 			(effects
@@
 			(project ""
 				(path "/b6a8d14b-6e32-4628-bf0c-2046877d1cfa/205555cc-3b86-4915-975e-3a7e3eed6661/84e3f5e1-ab68-44f3-8700-c3af58140fdb"
-					(reference "R20")
+					(reference "R16")
 					(unit 1)
 				)
@@
 		(dnp no)
 		(fields_autoplaced yes)
-		(property "Reference" "#PWR031"
+		(property "Reference" "#PWR032"
 			(at 243.84 124.46 0)
 			(effects
@@
 			(project "IMU_V100"
 				(path "/b6a8d14b-6e32-4628-bf0c-2046877d1cfa/205555cc-3b86-4915-975e-3a7e3eed6661/84e3f5e1-ab68-44f3-8700-c3af58140fdb"
-					(reference "#PWR031")
-					(unit 1)
-				)
+					(reference "#PWR032")
+					(unit 1)
+				)
